File: hardware/Motherboard/Video_CTRL.kicad_sch (KiCad schematic)
At the start: 0 parts

Commit message: WIP
Parts:
- added U56: 74LS541, symbol 74xx:74LS541
- added U59: EF9365, Package_DIP:DIP-40_W15.24mm, symbol parts:EF9365
- added U64: 74LS374, symbol 74xx:74LS374
Connections:
- new net: U59.1 (CK), U64.11 (Cp)
- new net: U59.25 (BLK), U64.13 (D4)
- new net: U59.14 (~{DW}), U64.14 (D5)
- new net: U59.15 (DIN), U64.17 (D6)
- new net: U59.6 (MSL0), U64.3 (D0)
- new net: U59.36 (MSL1), U64.4 (D1)
- new net: U59.7 (MSL2), U64.7 (D2)
- new net: U59.35 (MSL3), U64.8 (D3)
- new net DAD0: U56.8 (A6), U59.37 (DAD0)
- new net DAD1: U56.7 (A5), U59.39 (DAD1)
- new net DAD2: U56.6 (A4), U59.38 (DAD2)
- new net DAD3: U56.5 (A3), U59.4 (DAD3)
- new net DAD4: U56.4 (A2), U59.3 (DAD4)
- new net DAD5: U56.3 (A1), U59.2 (DAD5)
- new net DAD6: U56.2 (A0), U59.5 (DAD6)
- new net PA0: U59.9 (A0)
- new net PA1: U59.10 (A1)
- new net PA2: U59.11 (A2)
- new net PA3: U59.12 (A3)
- new net PD0: U59.33 (D0)
- new net PD1: U59.32 (D1)
- new net PD2: U59.31 (D2)
- new net PD3: U59.30 (D3)
- new net PD4: U59.29 (D4)
- new net PD5: U59.28 (D5)
- new net PD6: U59.27 (D6)
- new net PD7: U59.26 (D7)
- new net VA0: U56.12 (Y6)
- new net VA1: U56.13 (Y5)
- new net VA2: U56.14 (Y4)
- new net VA3: U56.15 (Y3)
- new net VA4: U56.16 (Y2)
- new net VA5: U56.17 (Y1)
- new net VA6: U56.18 (Y0)
- new net VCC5V: U56.20 (VCC), U59.40 (VCC), U64.20 (VCC)
- new net VSS: U56.1 (G1), U56.10 (GND), U56.19 (G2), U59.20 (VSS), U59.8 (FMAT), U64.1 (OE), U64.10 (GND)
- no-connect marks 0 -> 4

Commit message: WIP
Other:
- title: (none) -> Apollo 7 Squale - Video controller
Changed lines of the file:
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@@
 	(generator_version "9.0")
 	(paper "A4")
+	(title_block
+		(title "Apollo 7 Squale - Video controller")
+		(rev "0.1")
+		(comment 1 "http://hxc2001.free.fr/Squale/")
+		(comment 2 "CC-BY Licence (Creative Commons Attribution)")
+		(comment 3 "Drawn by Jean-François DEL NERO")
+	)
 	(junction
 		(at 171.45 127)

Commit message: WIP.
Parts:
- removed U56: 74LS541, symbol 74xx:74LS541
- removed U59: EF9365, Package_DIP:DIP-40_W15.24mm, symbol parts:EF9365
- removed U64: 74LS374, symbol 74xx:74LS374
Connections:
- no-connect marks 4 -> 0
