File: hardware/Motherboard/CPU.kicad_sch (KiCad schematic)
At the start: 9 parts, among them U1 MC6809, U10 74LS138, U2 27C64, U3 74LS245, U4 74LS139, U5 74LS20, U7 74LS02, U8 74LS00, U9 74LS541

Commit message: WIP
Other:
- note added: "0xF000 0xF010 0xF020 0xF030 0xF040 0xF050 0xF060 0xF070"
- note added: "0xFxxx"
- note added: "16 Bytes window per device. ~{CSES} Base : 0xF000"
- note added: "~{CSES} : 0xF000 - 0xF07F ~{CSS30} : 0xF080 - 0xF0FF ~{CSROM} : 0xF100 - 0xFFFF (Read only)"
Changed lines of the file:
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@@
 	(generator_version "9.0")
 	(paper "A3")
+	(text "0xF000\n0xF010\n0xF020\n0xF030\n0xF040\n0xF050\n0xF060\n0xF070"
+		(exclude_from_sim no)
+		(at 185.928 228.092 0)
+		(effects
+			(font
+				(size 1.651 1.651)
+			)
+		)
+	)
+	(text "0xFxxx"
+		(exclude_from_sim no)
+		(at 206.248 107.95 0)
+		(effects
+			(font
+				(size 1.27 1.27)
+			)
+		)
+	)
+	(text "16 Bytes window per device.\n~{CSES} Base : 0xF000"
+		(exclude_from_sim no)
+		(at 198.374 213.36 0)
+		(effects
+			(font
+				(size 1.651 1.651)
+			)
+		)
+	)
+	(text "~{CSES}  : 0xF000 - 0xF07F\n~{CSS30} : 0xF080 - 0xF0FF\n~{CSROM} : 0xF100 - 0xFFFF (Read only)"
+		(exclude_from_sim no)
+		(at 194.31 191.77 0)
+		(effects
+			(font
+				(size 1.651 1.651)
+			)
+			(justify left)
+		)
+	)
 	(junction
 		(at 166.37 101.6)

Commit message: WIP
Parts:
- removed unit 3 of U4
- added C16: 10uF 50V, symbol Device:C_Polarized
- added D3: 1N4148, Diode_THT:D_DO-35_SOD27_P7.62mm_Horizontal, symbol Diode:1N4148
- added R42: 10K, symbol Device:R
- added R43, R44, R45: 4.7K, symbol Device:R
- added unit 3 of U5
- added U6: 74LS08, symbol 74xx:74LS08
- added unit 5 of U8
Connections:
- net Q: now also U6.9
- net VCC5V: now also U1.33 (~{DMA/BREQ}), D3.1 (K), R42.1, R43.2, R44.2, R45.1, U5.14 (VCC), U6.1, U6.10, U6.14 (VCC), U8.14 (VCC)
- net VSS: now also U9.1 (G1), U9.19 (G2), C16.2, U5.7 (GND), U6.7 (GND), U8.7 (GND)
- net ~{CSES}: now also U6.4
- net ~{CSS30}: now also U6.5
- net R~{W}: now reaches U1.32 (R/~{W}), U5.1
- net R~{W}: now also U6.2
- net ~{NMI}: now reaches U1.2 (~{NMI})
- net ~{NMI}: now also R44.1
- net ~{IRQ}: now reaches U1.3 (~{IRQ})
- net ~{IRQ}: now also R43.1
- net ~{RST}: now reaches U1.37 (~{RESET})
- net ~{RST}: now also C16.1, D3.2 (A), R42.2
- net CLK_3.5MHz: now reaches U1.38 (EXTAL)
- net at U1.4 (~{FIRQ}): now also R45.2
- net R~{W}B: now reaches U3.1 (A->B)
- net R~{W}B: now also U6.3
- net at U3.19 (CE): now also U6.6
- new net QB: U6.8
- no-connect marks 6 -> 11
Other:
- moved on the sheet: U7A, U7B, U7C, U7D

Commit message: WIP
Connections:
- net VCC5V: now also R45.2; no longer R45.1
- net at U1.4 (~{FIRQ}): now also R45.1; no longer R45.2
Other:
- moved on the sheet: C16, D3, R42, R43, R44, R45

Commit message: WIP
Other:
- note added: "1 Machine cycle"
- note added: "10ns hold time (min)"
- note added: "1144nS / 874,126kHz"
- note added: "200ns max"
- note added: "286nS"
- note added: "80ns setup time (min)"
- note added: "E"
- note added: "Low -> 0xFxxx"
- note added: "Q"
- note added: "Read data"
- note added: "VMA"
- note added: "VMA = Valid Memory Address Start at the Q rising edge and end at the E falling edge"
- note added: "Valid Adresses, R~{W}, BS, BA"
- note added: "Valid Write data"
- note added: "XTAL 3.5MHz"
- note removed: "0xFxxx"
- title: (none) -> Apollo 7 Squale - CPU and decoders

Commit message: WIP
Other:
- note added: "Control signals"
- note added: "D (Read/In)"
- note added: "D (Write/Out)"
- moved on the sheet: C16, D3, R42, R43, R44, R45, U1, U10, U2, U3, U4A, U4B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

Commit message: WIP -rom pack
Parts:
- renumbered C16 to C5, D3 to D1, R42 to R20, R44 to R21, R43 to R23, R45 to R24, U6 to U10, U5 to U3, U8 to U4, U4 to U5, U10 to U6, U3 to U63, U9 to U64, U2 to U7, U7 to U9

Commit message: S30 bus + annotations fixes.
Parts:
- renumbered C5 to C16, D1 to D3, R20 to R42, R23 to R43, R21 to R44, R24 to R45, U6 to U10, U7 to U2, U63 to U3, U5 to U4, U3 to U5, U10 to U6, U9 to U7, U4 to U8, U64 to U9
Other:
- moved on the sheet: U5C, U6E, U7E, U8E
