File: hardware/Motherboard/CPU.kicad_sch (KiCad schematic)
At the start: 20 parts, among them U1 MC6809, U10 74LS138, U2 27C32, U3 74LS245, U4 74LS139, U5 74LS20, U6 74LS08, U66 74LS273, U7 74LS02, U8 74LS00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

Commit message: add some descriptions / comments.
Other:
- note added: "16 Bytes window per device. ~{CSES} Base address : 0xF000"
- note added: "Note : The V2.X Monitors need a 8kB 27C64 EPROM. In this case the extra EPROM A12 address line (pin 2) need to be connected with a wire to the U66 pin 19 output register (SYS_ROM_BK). The 27C64 pins 27, 28 and 1 need to be connected to the pin 26 (VCC5V)"
- note added: "Reset time : t = -log((V - Vc)/V)R*C = 161 ms With : V=5V (VCC5V) Vc=4V (Reset high level) R=10k (R42) C=10uF (C16)"
- note added: "System control register Base address : 0xF010"
- note removed: "16 Bytes window per device. ~{CSES} Base : 0xF000"
- note removed: "Note : The V2.X Monitors need a 27C64. In this case the extra EPROM A12 address line (pin 2) need to be connected with a wire to the U66 pin 19 output register (SYS_ROM_BK). The 27C64 pins 27, 28 and 1 need to be connected to the pin 26 (VCC5V)"
- note removed: "System control register Base :0xF010"
- moved on the sheet: D3, R42, U2
