File: hardware/Motherboard/sys_reg.kicad_sch (KiCad schematic)
At the start: 1 part, among them U66 74LS273

Commit message: wip : modem
Connections:
- net SYS_MDM_MC_~{BC}: now reaches U66.12 (Q4)
- net SYS_MDM_LINE: now reaches U66.15 (Q5)
- net SYS_KEYB_LED: now reaches U66.16 (Q6)
- net SYS_ROM_BK: now reaches U66.19 (Q7)
- net COL0 renamed SYS_COL0
- net COL1 renamed SYS_COL1
- net COL2 renamed SYS_COL2
- net COL3 renamed SYS_COL3
Changed lines of the file:
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@@
 	)
 	(bus_entry
-		(at 200.66 87.63)
+		(at 204.47 87.63)
 		(size 2.54 -2.54)
 		(stroke
@@
 	)
 	(bus_entry
-		(at 200.66 90.17)
+		(at 204.47 90.17)
 		(size 2.54 -2.54)
 		(stroke
@@
 	)
 	(bus_entry
-		(at 200.66 92.71)
+		(at 204.47 92.71)
 		(size 2.54 -2.54)
 		(stroke
@@
 	)
 	(bus_entry
-		(at 200.66 85.09)
+		(at 204.47 85.09)
 		(size 2.54 -2.54)
 		(stroke
@@
 		)
 	)
-	(bus
-		(pts
-			(xy 203.2 82.55) (xy 203.2 85.09)
+	(wire
+		(pts
+			(xy 193.04 100.33) (xy 227.33 100.33)
+		)
+		(stroke
+			(width 0)
+			(type default)
+		)
+	)
+	(bus
+		(pts
+			(xy 207.01 82.55) (xy 207.01 85.09)
+		)
+		(stroke
+			(width 0)
+			(type default)
+		)
+	)
+	(wire
+		(pts
+			(xy 193.04 85.09) (xy 204.47 85.09)
 		)
 		(stroke
@@
 	(bus
 		(pts
-			(xy 203.2 82.55) (xy 223.52 82.55)
+			(xy 207.01 82.55) (xy 227.33 82.55)
 		)
 		(stroke
@@
 		)
 	)
-	(bus
-		(pts
-			(xy 203.2 87.63) (xy 203.2 90.17)
+	(wire
+		(pts
+			(xy 193.04 102.87) (xy 227.33 102.87)
+		)
+		(stroke
+			(width 0)
+			(type default)
+		)
+	)
+	(bus
+		(pts
+			(xy 207.01 87.63) (xy 207.01 90.17)
 		)
 		(stroke
@@
 	(wire
 		(pts
-			(xy 193.04 92.71) (xy 200.66 92.71)
+			(xy 193.04 87.63) (xy 204.47 87.63)
 		)
 		(stroke
@@
 	(wire
 		(pts
+			(xy 193.04 95.25) (xy 227.33 95.25)
+		)
+		(stroke
+			(width 0)
+			(type default)
+		)
+	)
+	(wire
+		(pts
 			(xy 163.83 90.17) (xy 167.64 90.17)
 		)
@@
 	(wire
 		(pts
-			(xy 193.04 87.63) (xy 200.66 87.63)
+			(xy 193.04 92.71) (xy 204.47 92.71)
 		)
 		(stroke
@@
 	(wire
 		(pts
-			(xy 193.04 85.09) (xy 200.66 85.09)
-		)
-		(stroke
-			(width 0)
-			(type default)
-		)
-	)
-	(wire
-		(pts
 			(xy 163.83 102.87) (xy 167.64 102.87)
 		)
@@
 	(wire
 		(pts
-			(xy 193.04 90.17) (xy 200.66 90.17)
-		)
-		(stroke
-			(width 0)
-			(type default)
-		)
-	)
-	(bus
-		(pts
-			(xy 203.2 85.09) (xy 203.2 87.63)
+			(xy 193.04 90.17) (xy 204.47 90.17)
+		)
+		(stroke
+			(width 0)
+			(type default)
+		)
+	)
+	(bus
+		(pts
+			(xy 207.01 85.09) (xy 207.01 87.63)
 		)
 		(stroke
@@
 		(pts
 			(xy 76.2 110.49) (xy 167.64 110.49)
+		)
+		(stroke
+			(width 0)
+			(type default)
+		)
+	)
+	(wire
+		(pts
+			(xy 227.33 97.79) (xy 193.04 97.79)
 		)
 		(stroke
@@
 		)
 	)
-	(label "COL1"
+	(label "SYS_COL1"
 		(at 194.31 87.63 0)
 		(effects
@@
 		)
 	)
-	(label "COL3"
+	(label "SYS_COL3"
 		(at 194.31 92.71 0)
 		(effects
@@
 		)
 	)
-	(label "COL0"
+	(label "SYS_COL0"
 		(at 194.31 85.09 0)
 		(effects
@@
 		)
 	)
-	(label "COL2"
+	(label "SYS_COL2"
 		(at 194.31 90.17 0)
 		(effects
@@
 		)
 	)
+	(hierarchical_label "SYS_KEYB_LED"
+		(shape output)
+		(at 227.33 100.33 0)
+		(effects
+			(font
+				(size 1.27 1.27)
+			)
+			(justify left)
+		)
+	)
+	(hierarchical_label "SYS_MDM_LINE"
+		(shape output)
+		(at 227.33 97.79 0)
+		(effects
+			(font
+				(size 1.27 1.27)
+			)
+			(justify left)
+		)
+	)
 	(hierarchical_label "~{RSTB}"
 		(shape input)
@@
 		)
 	)
-	(hierarchical_label "COL[3..0]"
+	(hierarchical_label "SYS_COL[3..0]"
 		(shape output)
-		(at 223.52 82.55 0)
-		(effects
-			(font
+		(at 227.33 82.55 0)
+		(effects
+			(font
+				(size 1.27 1.27)
+			)
+			(justify left)
+		)
+	)
+	(hierarchical_label "SYS_MDM_MC_~{BC}"
+		(shape output)
+		(at 227.33 95.25 0)
+		(effects
+			(font
+				(size 1.27 1.27)
+			)
+			(justify left)
+		)
+	)
+	(hierarchical_label "SYS_ROM_BK"
+		(shape output)
+		(at 227.33 102.87 0)
+		(effects
+			(font
