File: hardware/Motherboard/sys_reg.kicad_sch (KiCad schematic)
At the start: 1 part, among them U66 74LS273

Commit message: WIP : passives parts, cosmetic stuffs.
Parts:
- removed U66: 74LS273, symbol 74xx:74LS273
