File: hardware/Motherboard/Video_RAM.kicad_sch (KiCad schematic)
At the start: 16 parts, among them U38 MK4116N, U39 MK4116N, U40 MK4116N, U42 MK4116N, U43 MK4116N, U44 MK4116N, U45 MK4116N, U46 MK4116N, U47 MK4116N, U48 MK4116N, U49 MK4116N, U50 MK4116N, U51 MK4116N, U52 MK4116N, U53 MK4116N

Commit message: WIP
Other:
- title: (none) -> Apollo 7 Squale - Video DRAM
Changed lines of the file:
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@@
 	(generator_version "9.0")
 	(paper "A3")
+	(title_block
+		(title "Apollo 7 Squale - Video DRAM")
+		(rev "0.1")
+		(comment 1 "http://hxc2001.free.fr/Squale/")
+		(comment 2 "CC-BY Licence (Creative Commons Attribution)")
+		(comment 3 "Drawn by Jean-François DEL NERO")
+	)
 	(text "Luminosité\nBrightness"
 		(exclude_from_sim no)

Commit message: WIP.
Parts:
- added U30, U31, U32, U33: 74LS166, symbol 74xx:74LS166
- added U56: 74LS541, symbol 74xx:74LS541
- added U59: EF9365, Package_DIP:DIP-40_W15.24mm, symbol parts:EF9365
- added U64: 74LS374, symbol 74xx:74LS374
Connections:
- net VA0: now also U56.12 (Y6)
- net VA1: now also U56.13 (Y5)
- net VA2: now also U56.14 (Y4)
- net VA3: now also U56.15 (Y3)
- net VA4: now also U56.16 (Y2)
- net VA5: now also U56.17 (Y1)
- net VA6: now also U56.18 (Y0)
- net VCC5V: now also U30.1 (Ds), U30.16 (VCC), U30.2 (A), U30.3 (B), U30.4 (C), U30.5 (D), U31.1 (Ds), U31.16 (VCC), U31.2 (A), U31.3 (B), U31.4 (C), U31.5 (D), U32.1 (Ds), U32.16 (VCC), U32.2 (A), U32.3 (B), U32.4 (C), U32.5 (D), U33.1 (Ds), U33.16 (VCC), U33.2 (A), U33.3 (B), U33.4 (C), U33.5 (D), U56.20 (VCC), U59.40 (VCC), U64.20 (VCC)
- net VSS: now also U30.8 (GND), U31.8 (GND), U32.8 (GND), U33.8 (GND), U56.1 (G1), U56.10 (GND), U56.19 (G2), U59.20 (VSS), U59.8 (FMAT), U64.1 (OE), U64.10 (GND)
- new net: U30.15 (PE), U31.15 (PE), U32.15 (PE), U33.15 (PE)
- new net: U30.6 (CE), U31.6 (CE), U32.6 (CE), U33.6 (CE)
- new net: U30.9 (Clr), U31.9 (Clr), U32.9 (Clr), U33.9 (Clr), U59.24 (~{WHITE})
- new net: U59.1 (CK), U64.11 (Cp)
- new net: U59.25 (BLK), U64.13 (D4)
- new net: U59.14 (~{DW}), U64.14 (D5)
- new net: U59.15 (DIN), U64.17 (D6)
- new net: U59.6 (MSL0), U64.3 (D0)
- new net: U59.36 (MSL1), U64.4 (D1)
- new net: U59.7 (MSL2), U64.7 (D2)
- new net: U59.35 (MSL3), U64.8 (D3)
- new net DAD0: U56.8 (A6), U59.37 (DAD0)
- new net DAD1: U56.7 (A5), U59.39 (DAD1)
- new net DAD2: U56.6 (A4), U59.38 (DAD2)
- new net DAD3: U56.5 (A3), U59.4 (DAD3)
- new net DAD4: U56.4 (A2), U59.3 (DAD4)
- new net DAD5: U56.3 (A1), U59.2 (DAD5)
- new net DAD6: U56.2 (A0), U59.5 (DAD6)
- new net PA0: U59.9 (A0)
- new net PA1: U59.10 (A1)
- new net PA2: U59.11 (A2)
- new net PA3: U59.12 (A3)
- new net PD0: U59.33 (D0)
- new net PD1: U59.32 (D1)
- new net PD2: U59.31 (D2)
- new net PD3: U59.30 (D3)
- new net PD4: U59.29 (D4)
- new net PD5: U59.28 (D5)
- new net PD6: U59.27 (D6)
- new net PD7: U59.26 (D7)
- new net R~{W}: U59.18 (R/~{W})
- new net ~{CS_9365}: U59.17 (E)
- new net ~{IRQ}: U59.13 (~{IRQ})
- no-connect marks 0 -> 5
Other:
- moved on the sheet: U38, U39, U40, U42, U43, U44, U45, U46, U47, U48, U49, U50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

Commit message: WIP
Parts:
- added J1: DA15_Socket, symbol Connector:DA15_Socket
- added Q1, Q2, Q3, Q4, Q5, Q6, Q7: 2N2222, Package_TO_SOT_THT:TO-18-3, symbol Transistor_BJT:2N2219
- added R1, R10, R13, R16, R18, R19, R4, R7: 1K, symbol Device:R
- added R12: 10K, symbol Device:R
- added R14, R2, R9: 330R, symbol Device:R
- added R15, R3, R46, R8: 220R, symbol Device:R
- added R17: 2K2, symbol Device:R
- added U25: 74LS74, symbol 74xx:74LS74
- added U32: 74LS04, symbol 74xx:74LS04
- added U33: 74LS17, symbol 74xx:74LS07
- added U54, U55, U58: 74LS374, symbol 74xx:74LS374
- added U57, U63: 74LS32, symbol 74xx:74LS32
- added U62: TBP18S030N, symbol 74xx:74LS374
- renumbered U30 to U34, U31 to U35, U32 to U36, U33 to U37, U39 to U41
Connections:
- net HRB: now also U63.3
- net HRI: now also U63.8
- net HRR: now also U63.6
- net HRV: now also U63.11
- net PD0: now also U54.2 (O0), U55.2 (O0)
- net PD1: now also U54.5 (O1), U55.5 (O1)
- net PD2: now also U54.6 (O2), U55.6 (O2)
- net PD3: now also U54.9 (O3), U55.9 (O3)
- net PD4: now also U54.12 (O4), U55.12 (O4)
- net PD5: now also U54.15 (O5), U55.15 (O5)
- net PD6: now also U54.16 (O6), U55.16 (O6)
- net PD7: now also U54.19 (O7), U55.19 (O7)
- net VCC12V: now also J1.6
- net VCC5V: now also J1.13 (P13), Q1.3 (C), Q2.3 (C), Q3.3 (C), Q4.3 (C), Q5.3 (C), Q6.3 (C), Q7.3 (C), R12.1, R17.1, R46.1, U25.1 (~{R}), U32.14 (VCC), U33.14 (VCC), U54.20 (VCC), U55.20 (VCC), U57.14 (VCC), U58.20 (VCC), U62.16 (VCC), U63.14 (VCC)
- net VSS: now also U59.23 (WO), J1.14 (P14), J1.15 (P15), R1.2, R10.2, R13.2, R15.2, R18.2, R19.2, R3.2, R8.2, U32.7 (GND), U33.7 (GND), U54.10 (GND), U55.10 (GND), U57.7 (GND), U58.1 (OE), U58.10 (GND), U62.15 (~{G}), U62.8 (GND), U63.7 (GND)
- net W0: now also U57.3
- net W1: now also U57.11
- net W2: now also U57.6
- net W3: now also U57.8
- net ~{D_{0}B}: now also U54.13 (D4)
- net ~{D_{0}I}: now also U54.18 (D7)
- net ~{D_{0}R}: now also U54.17 (D6)
- net ~{D_{0}V}: now also U54.14 (D5)
- net ~{D_{1}B}: now also U54.3 (D0)
- net ~{D_{1}I}: now also U54.8 (D3)
- net ~{D_{1}R}: now also U54.7 (D2)
- net ~{D_{1}V}: now also U54.4 (D1)
- net ~{D_{2}B}: now also U55.13 (D4)
- net ~{D_{2}I}: now also U55.18 (D7)
- net ~{D_{2}R}: now also U55.17 (D6)
- net ~{D_{2}V}: now also U55.14 (D5)
- net ~{D_{3}B}: now also U55.3 (D0)
- net ~{D_{3}I}: now also U55.8 (D3)
- net ~{D_{3}R}: now also U55.7 (D2)
- net ~{D_{3}V}: now also U55.4 (D1)
- net ~{VCAS}: now reaches U38.15 (~{CAS}), U39.15 (~{CAS}), U40.15 (~{CAS}), U41.15 (~{CAS}), U42.15 (~{CAS}), U43.15 (~{CAS}), U44.15 (~{CAS}), U45.15 (~{CAS}), U46.15 (~{CAS}), U47.15 (~{CAS}), U48.15 (~{CAS}), U49.15 (~{CAS}), U50.15 (~{CAS}), U51.15 (~{CAS}), U52.15 (~{CAS}), U53.15 (~{CAS})
- net ~{VCAS}: now also U58.5 (O1)
- net ~{VRAS}: now reaches U38.4 (~{RAS}), U39.4 (~{RAS}), U40.4 (~{RAS}), U41.4 (~{RAS}), U42.4 (~{RAS}), U43.4 (~{RAS}), U44.4 (~{RAS}), U45.4 (~{RAS}), U46.4 (~{RAS}), U47.4 (~{RAS}), U48.4 (~{RAS}), U49.4 (~{RAS}), U50.4 (~{RAS}), U51.4 (~{RAS}), U52.4 (~{RAS}), U53.4 (~{RAS})
- net ~{VRAS}: now also U58.6 (O2)
- net at U35.13 (Qh): now also U32.11
- net ~{VSHIFTLD}: now reaches U34.15 (PE), U35.15 (PE), U36.15 (PE), U37.15 (PE)
- net ~{VSHIFTLD}: now also U58.15 (O5)
- net CLK_7MHz: now reaches U34.6 (CE), U35.6 (CE), U36.6 (CE), U37.6 (CE)
- net CLK_7MHz: now also U62.10 (A0)
- net ~{WHITE}: now reaches U34.9 (Clr), U35.9 (Clr), U36.9 (Clr), U37.9 (Clr), U59.24 (~{WHITE})
- net at U37.13 (Qh): now also U32.5
- net CK_9365: now reaches U59.1 (CK), U64.11 (Cp)
- net CK_9365: now also U58.2 (O0)
- net BLKB: now reaches U64.12 (O4)
- net BLKB: now also U62.14 (A4)
- net BLK: now reaches U59.25 (BLK), U64.13 (D4)
- net ~{DW}: now reaches U59.14 (~{DW}), U64.14 (D5)
- net ~{DWB}: now reaches U64.15 (O5)
- net ~{DWB}: now also U62.13 (A3)
- net DINB: now reaches U64.16 (O6)
- net DINB: now also U63.10, U63.13, U63.2, U63.4
- net DIN: now reaches U59.15 (DIN), U64.17 (D6)
- net at U64.2 (O0): now also U57.1
- net at U64.5 (O1): now also U57.12
- net at U64.6 (O2): now also U57.5
- net at U64.9 (O3): no longer names the net of U64.9 (O3)
- net at U64.9 (O3): now also U57.9
- net at U36.13 (Qh): now also U32.9
- net ~{MFREE}: now reaches U59.19 (~{MFREE})
- net ~{MFREE}: now also U25.2 (D)
- net OpticalCK: now reaches U59.21 (LPCK)
- net SYNC: now reaches U59.34 (SYNC)
- net SYNC: now also U32.1
- net at U34.13 (Qh): now also R12.2, U32.13
- new net: R14.2, R15.1, U33.4
- new net: Q6.1 (E), R16.1
- new net: Q5.2 (B), R14.1, R16.2
- new net: Q7.2 (B), R17.2, R18.1, U33.6
- new net: J1.7, R46.2
- new net: Q3.2 (B), R7.2, R9.1
- new net: Q2.1 (E), R4.1
- new net: Q1.2 (B), R2.1, R4.2
- new net: R8.1, R9.2, U33.12
- new net: Q4.1 (E), R7.1
- new net: R2.2, R3.1, U33.2
- new net: U58.13 (D4), U62.5 (Q4)
- new net: U58.14 (D5), U62.6 (Q5)
- new net: U25.4 (~{S}), U58.16 (O6)
- new net: U58.17 (D6), U62.7 (Q6)
- new net: U58.18 (D7), U62.9 (Q7)
- new net: U58.3 (D0), U62.1 (Q0)
- new net: U58.4 (D1), U62.2 (Q1)
- new net: U58.7 (D2), U62.3 (Q2)
- new net: U58.8 (D3), U62.4 (Q3)
- new net: U25.3 (C), U58.9 (O3)
- new net ANA_B: J1.1, Q5.1 (E), R13.1
- new net ANA_G: J1.2, Q3.1 (E), R10.1
- new net ANA_R: J1.10 (P10), Q1.1 (E), R1.1
- new net ANA_SYNC: J1.9 (P9), Q7.1 (E), R19.1
- new net CLK_1.75MHz: U62.12 (A2)
- new net CLK_14MHz: U58.11 (Cp)
- new net CLK_3.5MHz: U62.11 (A1)
- new net COL0: U63.1
- new net COL1: U63.12
- new net COL2: U63.5
- new net COL3: U63.9
- new net SOUND_OUT: J1.8
- new net TTL_B: J1.11 (P111), Q6.2 (B), U32.6
- new net TTL_G: J1.4, Q4.2 (B), U32.8
- new net TTL_LUM: J1.5, U32.12, U33.1, U33.13, U33.3
- new net TTL_R: J1.12 (P12), Q2.2 (B), U32.10
- new net TTL_SYNC: J1.3, U32.2, U33.5
- new net UPD_RD_REG: U25.5 (Q), U54.11 (Cp), U55.11 (Cp)
- new net ~{CS_V1}: U54.1 (OE)
- new net ~{CS_V2}: U55.1 (OE)
- new net ~{VWEN}: U57.10, U57.13, U57.2, U57.4, U58.12 (O4)
- no-connect marks 5 -> 12
Other:
- note added: "Color value"
- note added: "Color write gates"
- note added: "DRAM access logic"
- note added: "DRAMs addresses buffer"
- note added: "Driver stage : 3 bits color + 1 global intensity bit 2 * 8 level colors (15 teints)"
- note added: "Memory readback flipflop"
- note added: "Memory readback registers 0xF020 and 0xF030 base address. Updated with the 0xF 9365 command."
- note added: "Shifters stage"
- note added: "Video DRAM Memory bank : 4 * 4 * 16384 bits = 32768 bytes 4 components (I,R,G,B). 4 bits access per component 16 bits access for the whole bank."
- note added: "write enable gates"
- title: Apollo 7 Squale - Video DRAM -> Apollo 7 Squale - Video
- moved on the sheet: U34, U35, U36, U37, U38, U39, U40, U41, U42, U43, U44, U45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

Commit message: WIP -rom pack
Parts:
- renumbered Q2 to Q1, Q4 to Q2, Q6 to Q3, Q7 to Q4, Q1 to Q5, Q3 to Q6, Q5 to Q7, R12 to R1, R16 to R10, R14 to R11, R15 to R12, R17 to R13, R18 to R14, R19 to R15, R1 to R16, R10 to R17, R13 to R18, R46 to R19, R4 to R2, R2 to R3, R3 to R4, R9 to R8, R8 to R9, U33 to U30, U62 to U32, U54 to U33, U55 to U34, U59 to U35, U57 to U36, U58 to U37, U63 to U38, U64 to U39, U56 to U40, U32 to U41, U50 to U42, U51 to U43, U52 to U44, U53 to U45, U42 to U50, U43 to U51, U44 to U52, U45 to U53, U38 to U54, U39 to U55, U41 to U56, U40 to U57, U34 to U58, U35 to U59, U36 to U61, U37 to U62

Commit message: wip
Parts:
- renumbered U38 to U63
Changed lines of the file:
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@@
 		(on_board yes)
 		(dnp no)
-		(property "Reference" "U38"
+		(property "Reference" "U63"
 			(at 170.18 180.34 0)
 			(effects
@@
 			(project "Squale"
 				(path "/9e981419-a202-4dd8-b7ec-e1bde8e7b185/64986b08-7b2b-4504-b87f-fa7d0c749ced"
-					(reference "U38")
+					(reference "U63")
 					(unit 1)
 				)
@@
 		(dnp no)
 		(fields_autoplaced yes)
-		(property "Reference" "U38"
+		(property "Reference" "U63"
 			(at 121.92 346.7099 0)
 			(effects
@@
 			(project "Squale"
 				(path "/9e981419-a202-4dd8-b7ec-e1bde8e7b185/64986b08-7b2b-4504-b87f-fa7d0c749ced"
-					(reference "U38")
+					(reference "U63")
 					(unit 5)
 				)
@@
 		(on_board yes)
 		(dnp no)
-		(property "Reference" "U38"
+		(property "Reference" "U63"
 			(at 170.434 160.02 0)
 			(effects
@@
 			(project "Squale"
 				(path "/9e981419-a202-4dd8-b7ec-e1bde8e7b185/64986b08-7b2b-4504-b87f-fa7d0c749ced"
-					(reference "U38")
+					(reference "U63")
 					(unit 2)
 				)
@@
 		(on_board yes)
 		(dnp no)
-		(property "Reference" "U38"
+		(property "Reference" "U63"
 			(at 169.926 149.606 0)
 			(effects
@@
 			(project "Squale"
 				(path "/9e981419-a202-4dd8-b7ec-e1bde8e7b185/64986b08-7b2b-4504-b87f-fa7d0c749ced"
-					(reference "U38")
+					(reference "U63")
 					(unit 3)
 				)
@@
 		(on_board yes)
 		(dnp no)
-		(property "Reference" "U38"
+		(property "Reference" "U63"
 			(at 170.18 170.18 0)
 			(effects
@@
 			(project "Squale"
 				(path "/9e981419-a202-4dd8-b7ec-e1bde8e7b185/64986b08-7b2b-4504-b87f-fa7d0c749ced"
-					(reference "U38")
+					(reference "U63")
 					(unit 4)
 				)

Commit message: S30 bus + annotations fixes.
Parts:
- renumbered Q5 to Q1, Q1 to Q2, Q6 to Q3, Q2 to Q4, Q7 to Q5, Q3 to Q6, Q4 to Q7, R16 to R1, R17 to R10, R1 to R12, R18 to R13, R11 to R14, R12 to R15, R10 to R16, R13 to R17, R14 to R18, R15 to R19, R3 to R2, R4 to R3, R2 to R4, R19 to R46, R9 to R8, R8 to R9, U41 to U32, U30 to U33, U58 to U34, U59 to U35, U61 to U36, U62 to U37, U54 to U38, U55 to U39, U56 to U40, U57 to U41, U50 to U42, U51 to U43, U52 to U44, U53 to U45, U42 to U50, U43 to U51, U44 to U52, U45 to U53, U33 to U54, U34 to U55, U40 to U56, U36 to U57, U37 to U58, U35 to U59, U32 to U62, U39 to U64

Commit message: wip : modem
Connections:
- net COL0 renamed SYS_COL0
- net COL1 renamed SYS_COL1
- net COL2 renamed SYS_COL2
- net COL3 renamed SYS_COL3
Other:
- moved on the sheet: U63A, U63B, U63C, U63D
Changed lines of the file:
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@@
 	(wire
 		(pts
-			(xy 181.61 171.45) (xy 203.2 171.45)
+			(xy 185.42 171.45) (xy 203.2 171.45)
 		)
 		(stroke
@@
 	(wire
 		(pts
-			(xy 181.61 175.26) (xy 181.61 171.45)
+			(xy 185.42 175.26) (xy 185.42 171.45)
 		)
 		(stroke
@@
 	(wire
 		(pts
-			(xy 162.56 152.4) (xy 166.37 152.4)
+			(xy 162.56 152.4) (xy 170.18 152.4)
 		)
 		(stroke
@@
 	(wire
 		(pts
-			(xy 157.48 157.48) (xy 166.37 157.48)
+			(xy 157.48 157.48) (xy 170.18 157.48)
 		)
 		(stroke
@@
 	(wire
 		(pts
-			(xy 162.56 172.72) (xy 166.37 172.72)
+			(xy 162.56 172.72) (xy 170.18 172.72)
 		)
 		(stroke
@@
 	(wire
 		(pts
-			(xy 166.37 187.96) (xy 157.48 187.96)
+			(xy 170.18 187.96) (xy 157.48 187.96)
 		)
 		(stroke
@@
 	(wire
 		(pts
-			(xy 157.48 177.8) (xy 166.37 177.8)
+			(xy 157.48 177.8) (xy 170.18 177.8)
 		)
 		(stroke
@@
 	(wire
 		(pts
-			(xy 162.56 162.56) (xy 166.37 162.56)
+			(xy 162.56 162.56) (xy 170.18 162.56)
 		)
 		(stroke
@@
 	(wire
 		(pts
-			(xy 157.48 167.64) (xy 166.37 167.64)
+			(xy 157.48 167.64) (xy 170.18 167.64)
 		)
 		(stroke
@@
 	(wire
 		(pts
-			(xy 181.61 165.1) (xy 198.12 165.1)
+			(xy 185.42 165.1) (xy 198.12 165.1)
 		)
 		(stroke
@@
 	(wire
 		(pts
-			(xy 181.61 185.42) (xy 187.96 185.42)
+			(xy 185.42 185.42) (xy 187.96 185.42)
 		)
 		(stroke
@@
 	(wire
 		(pts
-			(xy 162.56 182.88) (xy 166.37 182.88)
+			(xy 162.56 182.88) (xy 170.18 182.88)
 		)
 		(stroke
@@
 	(wire
 		(pts
-			(xy 181.61 154.94) (xy 195.58 154.94)
-		)
-		(stroke
-			(width 0)
-			(type default)
-		)
-	)
-	(wire
-		(pts
 			(xy 58.42 54.61) (xy 59.69 54.61)
 		)
@@
 	(wire
 		(pts
+			(xy 185.42 154.94) (xy 195.58 154.94)
+		)
+		(stroke
+			(width 0)
+			(type default)
+		)
+	)
+	(wire
+		(pts
 			(xy 539.75 139.7) (xy 539.75 261.62)
 		)
@@
 		)
 	)
-	(label "COL2"
+	(label "SYS_COL2"
 		(at 162.56 162.56 0)
 		(effects
@@
 		)
 	)
-	(label "COL0"
+	(label "SYS_COL0"
 		(at 162.56 182.88 0)
 		(effects
@@
 	)
 	(label "HRB"
-		(at 182.88 185.42 0)
+		(at 185.42 185.42 0)
 		(effects
 			(font
@@
 	)
 	(label "HRV"
-		(at 182.88 171.45 0)
+		(at 185.42 171.45 0)
 		(effects
 			(font
@@
 		)
 	)
-	(label "COL3"
+	(label "SYS_COL3"
 		(at 162.56 152.4 0)
 		(effects
@@
 	)
 	(label "HRI"
-		(at 182.88 154.94 0)
+		(at 185.42 154.94 0)
 		(effects
 			(font
@@
 		)
 	)
-	(label "COL1"
+	(label "SYS_COL1"
 		(at 162.56 172.72 0)
 		(effects
@@
 		)
 	)
-	(label "COL[3..0]"
+	(label "SYS_COL[3..0]"
 		(at 95.25 204.47 0)
 		(effects
@@
 	)
 	(label "HRR"
-		(at 182.88 165.1 0)
+		(at 185.42 165.1 0)
 		(effects
 			(font
@@
 		)
 	)
-	(hierarchical_label "COL[3..0]"
+	(hierarchical_label "SYS_COL[3..0]"
 		(shape input)
 		(at 43.18 204.47 180)
@@
 	(symbol
 		(lib_id "74xx:74LS32")
-		(at 173.99 185.42 0)
+		(at 177.8 185.42 0)
 		(unit 1)
 		(exclude_from_sim no)
@@
 		(dnp no)
 		(property "Reference" "U63"
-			(at 170.18 180.34 0)
+			(at 173.99 180.34 0)
 			(effects
 				(font
@@
 		)
 		(property "Value" "74LS32"
-			(at 176.784 180.34 0)
+			(at 180.594 180.34 0)
 			(effects
 				(font
@@
 		)
 		(property "Footprint" ""
-			(at 173.99 185.42 0)
+			(at 177.8 185.42 0)
 			(effects
 				(font
@@
 		)
 		(property "Datasheet" "http://www.ti.com/lit/gpn/sn74LS32"
-			(at 173.99 185.42 0)
+			(at 177.8 185.42 0)
 			(effects
 				(font
@@
 		)
 		(property "Description" "Quad 2-input OR"
-			(at 173.99 185.42 0)
+			(at 177.8 185.42 0)
 			(effects
 				(font
@@
 	(symbol
 		(lib_id "74xx:74LS32")
-		(at 173.99 165.1 0)
+		(at 177.8 165.1 0)
 		(mirror x)
 		(unit 2)
@@
 		(dnp no)
 		(property "Reference" "U63"
-			(at 170.434 160.02 0)
+			(at 174.244 160.02 0)
 			(effects
 				(font
@@
 		)
 		(property "Value" "74LS32"
-			(at 177.038 160.02 0)
+			(at 180.848 160.02 0)
 			(effects
 				(font
@@
 		)
 		(property "Footprint" ""
-			(at 173.99 165.1 0)
+			(at 177.8 165.1 0)
 			(effects
 				(font
@@
 		)
 		(property "Datasheet" "http://www.ti.com/lit/gpn/sn74LS32"
-			(at 173.99 165.1 0)
+			(at 177.8 165.1 0)
 			(effects
 				(font
@@
 		)
 		(property "Description" "Quad 2-input OR"
-			(at 173.99 165.1 0)
+			(at 177.8 165.1 0)
 			(effects
 				(font
@@
 	(symbol
 		(lib_id "74xx:74LS32")
-		(at 173.99 154.94 0)
+		(at 177.8 154.94 0)
 		(unit 3)
 		(exclude_from_sim no)
@@
 		(dnp no)
 		(property "Reference" "U63"
-			(at 169.926 149.606 0)
+			(at 173.736 149.606 0)
 			(effects
 				(font
@@
 		)
 		(property "Value" "74LS32"
-			(at 177.038 149.606 0)
+			(at 180.848 149.606 0)
 			(effects
 				(font
@@
 		)
 		(property "Footprint" ""
-			(at 173.99 154.94 0)
+			(at 177.8 154.94 0)
 			(effects
 				(font
@@
 		)
 		(property "Datasheet" "http://www.ti.com/lit/gpn/sn74LS32"
-			(at 173.99 154.94 0)
+			(at 177.8 154.94 0)
 			(effects
 				(font
@@
 		)
 		(property "Description" "Quad 2-input OR"
-			(at 173.99 154.94 0)
+			(at 177.8 154.94 0)
 			(effects
 				(font
@@
 	(symbol
 		(lib_id "74xx:74LS32")
-		(at 173.99 175.26 0)
+		(at 177.8 175.26 0)
 		(unit 4)
 		(exclude_from_sim no)
@@
 		(dnp no)
 		(property "Reference" "U63"
-			(at 170.18 170.18 0)
+			(at 173.99 170.18 0)
 			(effects
 				(font
@@
 		)
 		(property "Value" "74LS32"
-			(at 176.784 170.18 0)
+			(at 180.594 170.18 0)
 			(effects
 				(font
@@
 		)
 		(property "Footprint" ""
-			(at 173.99 175.26 0)
+			(at 177.8 175.26 0)
 			(effects
 				(font
@@
 		)
 		(property "Datasheet" "http://www.ti.com/lit/gpn/sn74LS32"
-			(at 173.99 175.26 0)
+			(at 177.8 175.26 0)
 			(effects
 				(font
@@
 		)
 		(property "Description" "Quad 2-input OR"
-			(at 173.99 175.26 0)
+			(at 177.8 175.26 0)
 			(effects
 				(font

Commit message: wip
Parts:
- added J9: DIN-5_180degree, symbol Connector:DIN-5_180degree
- added R41: 10K, symbol Device:R
Connections:
- net VCC5V: now also J9.1, R41.1
- net VSS: now also J9.2
- net OpticalCK renamed LIGHTPEN_STROBE
- net LIGHTPEN_STROBE: now also J9.5, R41.2
- new net LIGHTPEN_SWITCH: J9.3
- no-connect marks 12 -> 13
Other:
- moved on the sheet: U32B, U33E
