File: hardware/Motherboard/tape_modem.kicad_sch (KiCad schematic)
At the start: 34 parts, among them J5 DIN-5_180degree, J6 DE9_Socket, P1 VR10K, U67 TL084, U68 EFB7510, U69 MC6850, U70 74LS02, U71 74LS393, Y2 3.579MHz

Commit message: wip
Changed lines of the file:
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@@
 	(text "max level :\n+8 dBm (< 6 VPP)"
 		(exclude_from_sim no)
-		(at 272.796 108.458 0)
+		(at 272.034 110.744 0)
 		(effects
 			(font
@@
 	(wire
 		(pts
-			(xy 373.38 83.82) (xy 373.38 146.05)
+			(xy 375.92 87.63) (xy 375.92 146.05)
 		)
 		(stroke
@@
 	(polyline
 		(pts
-			(xy 271.78 95.25) (xy 372.11 95.25)
+			(xy 271.78 95.25) (xy 373.38 95.25)
 		)
 		(stroke
@@
 	(polyline
 		(pts
-			(xy 372.11 95.25) (xy 372.11 186.69)
+			(xy 373.38 95.25) (xy 373.38 186.69)
 		)
 		(stroke
@@
 	(wire
 		(pts
-			(xy 300.99 83.82) (xy 373.38 83.82)
+			(xy 300.99 87.63) (xy 375.92 87.63)
 		)
 		(stroke
@@
 	(wire
 		(pts
-			(xy 300.99 59.69) (xy 300.99 83.82)
+			(xy 300.99 59.69) (xy 300.99 87.63)
 		)
 		(stroke
@@
 	(wire
 		(pts
-			(xy 393.7 146.05) (xy 373.38 146.05)
+			(xy 393.7 146.05) (xy 375.92 146.05)
 		)
 		(stroke
@@
 	(polyline
 		(pts
-			(xy 372.11 186.69) (xy 279.4 186.69)
+			(xy 373.38 186.69) (xy 279.4 186.69)
 		)
 		(stroke
@@
 	(polyline
 		(pts
-			(xy 279.4 185.42) (xy 279.4 123.19)
+			(xy 279.4 186.69) (xy 279.4 123.19)
 		)
 		(stroke
@@
 	(polyline
 		(pts
-			(xy 279.4 185.42) (xy 279.4 185.42)
-		)
-		(stroke
+			(xy 279.4 186.69) (xy 279.4 185.42)
+		)
+		(stroke
