File: hardware/Motherboard/DRAM.kicad_sch (KiCad schematic)
At the start: 25 parts, among them U11 74LS245, U12 74LS541, U13 74LS541, U14 74LS541, U15 74LS393, U16 MK4164N, U17 MK4164N, U18 MK4164N, U19 MK4164N, U2 74LS123, U20 MK4164N, U21 MK4164N, U22 MK4164N, U23 MK4164N, U24 74LS123, U25 74LS74, U26 74LS74, U28 74LS04, U29 74LS02, U8 74LS00

Commit message: WIP
Parts:
- renumbered C3 to C28, C2 to C3, C1 to C4, R1 to R22, R2 to R48
Connections:
- net QB: now reaches U28.1
- net PRW renamed R~{W}B
Changed lines of the file:
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@@
 		)
 	)
-	(label "PRW"
+	(label "R~{W}B"
 		(at 177.8 274.32 0)
 		(effects
@@
 		)
 	)
+	(label "QB"
+		(at 16.51 248.92 0)
+		(effects
+			(font
+				(size 1.27 1.27)
+			)
+			(justify left bottom)
+		)
+	)
 	(label "VMA"
 		(at 207.01 167.64 0)
@@
 		(dnp no)
 		(fields_autoplaced yes)
-		(property "Reference" "R2"
+		(property "Reference" "R48"
 			(at 95.25 190.4999 0)
 			(effects
@@
 			(project "Squale"
 				(path "/9e981419-a202-4dd8-b7ec-e1bde8e7b185/7d7f151b-a16e-4418-bf6d-71f4cdd2beb8"
-					(reference "R2")
+					(reference "R48")
 					(unit 1)
 				)
@@
 		(dnp no)
 		(fields_autoplaced yes)
-		(property "Reference" "R1"
+		(property "Reference" "R22"
 			(at 95.25 231.1399 0)
 			(effects
@@
 			(project "Squale"
 				(path "/9e981419-a202-4dd8-b7ec-e1bde8e7b185/7d7f151b-a16e-4418-bf6d-71f4cdd2beb8"
-					(reference "R1")
+					(reference "R22")
 					(unit 1)
 				)
@@
 		(dnp no)
 		(fields_autoplaced yes)
-		(property "Reference" "C3"
+		(property "Reference" "C28"
 			(at 81.28 252.7299 0)
 			(effects
@@
 			(project "Squale"
 				(path "/9e981419-a202-4dd8-b7ec-e1bde8e7b185/7d7f151b-a16e-4418-bf6d-71f4cdd2beb8"
-					(reference "C3")
+					(reference "C28")
 					(unit 1)
 				)
@@
 		(dnp no)
 		(fields_autoplaced yes)
-		(property "Reference" "C2"
+		(property "Reference" "C3"
 			(at 96.52 198.1199 0)
 			(effects
@@
 			(project "Squale"
 				(path "/9e981419-a202-4dd8-b7ec-e1bde8e7b185/7d7f151b-a16e-4418-bf6d-71f4cdd2beb8"
-					(reference "C2")
+					(reference "C3")
 					(unit 1)
 				)
@@
 		(dnp no)
 		(fields_autoplaced yes)
-		(property "Reference" "C1"
+		(property "Reference" "C4"
 			(at 96.52 238.7599 0)
 			(effects
@@
 			(project "Squale"
 				(path "/9e981419-a202-4dd8-b7ec-e1bde8e7b185/7d7f151b-a16e-4418-bf6d-71f4cdd2beb8"
-					(reference "C1")
+					(reference "C4")
 					(unit 1)
 				)

Commit message: WIP.
Parts:
- removed unit 3 of U29
- removed unit 2 of U29
Changed lines of the file:
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@@
 	)
 	(symbol
-		(lib_id "74xx:74LS02")
-		(at 210.82 194.31 0)
-		(unit 3)
-		(exclude_from_sim no)
-		(in_bom yes)
-		(on_board yes)
-		(dnp no)
-		(fields_autoplaced yes)
-		(property "Reference" "U29"
-			(at 210.82 185.42 0)
-			(effects
-				(font
-					(size 1.27 1.27)
-				)
-			)
-		)
-		(property "Value" "74LS02"
-			(at 210.82 187.96 0)
-			(effects
-				(font
-					(size 1.27 1.27)
-				)
-			)
-		)
-		(property "Footprint" ""
-			(at 210.82 194.31 0)
-			(effects
-				(font
-					(size 1.27 1.27)
-				)
-				(hide yes)
-			)
-		)
-		(property "Datasheet" "http://www.ti.com/lit/gpn/sn74ls02"
-			(at 210.82 194.31 0)
-			(effects
-				(font
-					(size 1.27 1.27)
-				)
-				(hide yes)
-			)
-		)
-		(property "Description" "quad 2-input NOR gate"
-			(at 210.82 194.31 0)
-			(effects
-				(font
-					(size 1.27 1.27)
-				)
-				(hide yes)
-			)
-		)
-		(pin "14"
-		)
-		(pin "12"
-		)
-		(pin "1"
-		)
-		(pin "3"
-		)
-		(pin "9"
-		)
-		(pin "10"
-		)
-		(pin "6"
-		)
-		(pin "7"
-		)
-		(pin "13"
-		)
-		(pin "11"
-		)
-		(pin "4"
-		)
-		(pin "8"
-		)
-		(pin "2"
-		)
-		(pin "5"
-		)
-		(instances
-			(project "Squale"
-				(path "/9e981419-a202-4dd8-b7ec-e1bde8e7b185/7d7f151b-a16e-4418-bf6d-71f4cdd2beb8"
-					(reference "U29")
-					(unit 3)
-				)
-			)
-		)
-	)
-	(symbol
 		(lib_id "Device:R")
 		(at 92.71 191.77 0)
@@
 				)
 			)
-		)
-	)
-	(symbol
-		(lib_id "74xx:74LS02")
-		(at 232.41 193.04 0)
-		(unit 2)
-		(exclude_from_sim no)
-		(in_bom yes)
-		(on_board yes)
-		(dnp no)
-		(fields_autoplaced yes)
-		(property "Reference" "U29"
-			(at 232.41 184.15 0)
-			(effects
-				(font
-					(size 1.27 1.27)
-				)
-			)
-		)
-		(property "Value" "74LS02"
-			(at 232.41 186.69 0)
-			(effects
-				(font
-					(size 1.27 1.27)
-				)
-			)
-		)
-		(property "Footprint" ""
-			(at 232.41 193.04 0)
-			(effects
-				(font
-					(size 1.27 1.27)
-				)
-				(hide yes)
-			)
-		)
-		(property "Datasheet" "http://www.ti.com/lit/gpn/sn74ls02"
-			(at 232.41 193.04 0)
-			(effects
-				(font
-					(size 1.27 1.27)
-				)
-				(hide yes)
-			)
-		)
-		(property "Description" "quad 2-input NOR gate"
-			(at 232.41 193.04 0)
-			(effects
-				(font
-					(size 1.27 1.27)
-				)
-				(hide yes)
-			)
-		)
-		(pin "14"
-		)
-		(pin "12"
-		)
-		(pin "1"
-		)
-		(pin "3"
-		)
-		(pin "9"
-		)
-		(pin "10"
-		)
-		(pin "6"
-		)
-		(pin "7"
-		)
-		(pin "13"
-		)
-		(pin "11"
-		)
-		(pin "4"
-		)
-		(pin "8"
-		)
-		(pin "2"
-		)
-		(pin "5"
-		)
-		(instances
-			(project "Squale"
-				(path "/9e981419-a202-4dd8-b7ec-e1bde8e7b185/7d7f151b-a16e-4418-bf6d-71f4cdd2beb8"
-					(reference "U29")
-					(unit 2)
-				)
-			)

Commit message: WIP
Parts:
- removed unit 1 of U25
- added U71: 74LS393, symbol 74xx:74LS393
Connections:
- net EB: now also U71.13 (CP)
- net R~{W}B: now also U11.1 (A->B)
- net VSS: now also U71.12 (MR)
- net at U24.1 (A): now also U71.9 (Q2)
- net ~{DatEn}: now reaches U28.13, U8.3
- net ~{DatEn}: now also U11.19 (CE)
- no-connect marks 12 -> 15
Other:
- note added: "1 Machine cycle"
- note added: "109,373kHz"
- note added: "10ns hold time (min)"
- note added: "1144nS / 874,126kHz"
- note added: "200ns max"
- note added: "286nS"
- note added: "80ns setup time (min)"
- note added: "9,144 us refresh period * 256 = 2.34 ms total DRAM refresh period."
- note added: "CAS address buffer (A15-A8)"
- note added: "CPU Bus"
- note added: "Colon Address (A15-A8)"
- note added: "Control signals"
- note added: "D (In/read)"
- note added: "D (Write/Out)"
- note added: "DRAM A7-A0"
- note added: "DRAM Controller"
- note added: "DRAM Read/Write cycle : 1 - ~{RAS} falling edge : Latch the row address 2 - ~{CAS} falling edge : Latch the column address and: Do a write operation if ~{WE} is low Do a read operation if ~{WE} is high"
- note added: "DRAM Refresh ( ~{RAS} only refresh ): 1 - ~{RAS} falling edge : Latch the row address 2 - ~{RAS} rising edge : Do the row refresh"
- note added: "DRAM Refresh / Read or Write access cycle"
- note added: "DRAM Refresh signal generator"
- note added: "DRAM refresh row address buffer"
- note added: "DRAM refresh row address counter"
- note added: "Data buffer (D7-D0)"
- note added: "E"
- note added: "End delay (Q rising + gates delay + ~24ns)"
- note added: "Memory access operation gates"
- note added: "Pre delay (E falling + counter delay + ~24ns)"
- note added: "Q"
- note added: "RAS Refresh cycle 9,144 us period"
- note added: "RAS address buffer (A7-A0)"
- note added: "Read data"
- note added: "Refresh Address"
- note added: "Row Address (A7-A0)"
- note added: "S2"
- note added: "VMA"
- note added: "Valid Adresses, R~{W}, BS, BA"
- note added: "Valid Write data"
- note added: "XTAL 3.5MHz"
- note added: "cycle machine clock divisor"
- note added: "~{CAS}"
- note added: "~{DatEn}"
- note added: "~{MUIH}"
- note added: "~{MUIL}"
- note added: "~{RAS}"
- note added: "~{RAS} only refresh or normal access ~{RAS}"
- note added: "~{RAS}/~{CAS} buffer address selector"
- note added: "~{WE}"
- note added: "~{WE} enabled (if needed) during the access period."
- note removed: "~24ns"
- title: (none) -> Apollo 7 Squale - DRAM controller
- moved on the sheet: U28B, U28C, U29D, U8A

Commit message: typo.
Other:
- note added: "Column Address (A15-A8)"
- note added: "D (Read/In)"
- note added: "Valid Address, R~{W}, BS, BA"
- note removed: "Colon Address (A15-A8)"
- note removed: "D (In/read)"
- note removed: "Valid Adresses, R~{W}, BS, BA"
- title: Apollo 7 Squale - DRAM controller -> Apollo 7 Squale - DRAM controller and 64KB of DRAM 
Changed lines of the file:
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@@
 	(paper "A3")
 	(title_block
-		(title "Apollo 7 Squale - DRAM controller")
+		(title "Apollo 7 Squale - DRAM controller and 64KB of DRAM ")
 		(date "2025-08-24")
 		(rev "0.1")
@@
 		)
 	)
-	(text "Colon\nAddress\n(A15-A8)"
+	(text "Column\nAddress\n(A15-A8)"
 		(exclude_from_sim no)
 		(at 231.394 122.682 0)
@@
 		)
 	)
-	(text "Valid Adresses,\nR~{W}, BS, BA"
+	(text "Valid Address,\nR~{W}, BS, BA"
 		(exclude_from_sim no)
 		(at 228.6 62.992 0)
@@
 		)
 	)
-	(text "D\n(In/read)"
+	(text "D\n(Read/In)"
 		(exclude_from_sim no)
 		(at 188.976 78.486 0)
@@
 		)
 	)
-	(text "Colon\nAddress\n(A15-A8)"
+	(text "Column\nAddress\n(A15-A8)"
 		(exclude_from_sim no)
 		(at 202.184 122.682 0)

Commit message: WIP -rom pack
Other:
- moved on the sheet: C28, C3, C4, R22, R48, U15C, U24A, U24B, U25B, U25C, U26A, U26C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

Commit message: wip
Parts:
- added U7: 74LS02, symbol 74xx:74LS02
Connections:
- net VMA: now also U7.13
- net ~{VMA}: now also U7.11, U7.12
Other:
- note added: "machine cycle clock divisor ( / 8 )"
- note removed: "cycle machine clock divisor"
Changed lines of the file:
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@@
 		)
 	)
-	(text "cycle machine \nclock divisor"
+	(text "machine cycle \nclock divisor\n( / 8 )\n"
 		(exclude_from_sim no)
 		(at 65.278 220.218 0)
@@
 	)
 	(junction
+		(at 35.56 190.5)
+		(diameter 0)
+		(color 0 0 0 0)
+	)
+	(junction
 		(at 389.89 97.79)
 		(diameter 0)
@@
 	)
 	(junction
+		(at 31.75 190.5)
+		(diameter 0)
+		(color 0 0 0 0)
+	)
+	(junction
 		(at 389.89 201.93)
 		(diameter 0)
@@
 	(wire
 		(pts
+			(xy 81.28 167.64) (xy 116.84 167.64)
+		)
+		(stroke
+			(width 0)
+			(type default)
+		)
+	)
+	(wire
+		(pts
 			(xy 278.13 157.48) (xy 281.94 157.48)
 		)
@@
 	(wire
 		(pts
+			(xy 53.34 190.5) (xy 72.39 190.5)
+		)
+		(stroke
+			(width 0)
+			(type default)
+		)
+	)
+	(wire
+		(pts
 			(xy 123.19 170.18) (xy 129.54 170.18)
 		)
@@
 		)
 	)
+	(wire
+		(pts
+			(xy 38.1 193.04) (xy 35.56 193.04)
+		)
+		(stroke
+			(width 0)
+			(type default)
+		)
+	)
 	(polyline
 		(pts
@@
 		)
 	)
+	(wire
+		(pts
+			(xy 35.56 193.04) (xy 35.56 190.5)
+		)
+		(stroke
+			(width 0)
+			(type default)
+		)
+	)
 	(polyline
 		(pts
@@
 	(wire
 		(pts
-			(xy 107.95 167.64) (xy 116.84 167.64)
-		)
-		(stroke
-			(width 0)
-			(type default)
-		)
-	)
-	(wire
-		(pts
 			(xy 278.13 204.47) (xy 281.94 204.47)
 		)
@@
 	(wire
 		(pts
+			(xy 31.75 179.07) (xy 81.28 179.07)
+		)
+		(stroke
+			(width 0)
+			(type default)
+		)
+	)
+	(wire
+		(pts
 			(xy 278.13 102.87) (xy 281.94 102.87)
 		)
@@
 	(wire
 		(pts
+			(xy 35.56 190.5) (xy 35.56 187.96)
+		)
+		(stroke
+			(width 0)
+			(type default)
+		)
+	)
+	(wire
+		(pts
 			(xy 307.34 152.4) (xy 330.2 152.4)
 		)
@@
 		)
 	)
+	(wire
+		(pts
+			(xy 31.75 190.5) (xy 31.75 179.07)
+		)
+		(stroke
+			(width 0)
+			(type default)
+		)
+	)
 	(bus
 		(pts
@@
 	(wire
 		(pts
+			(xy 31.75 190.5) (xy 35.56 190.5)
+		)
+		(stroke
+			(width 0)
+			(type default)
+		)
+	)
+	(wire
+		(pts
 			(xy 227.33 161.29) (xy 227.33 152.4)
 		)
@@
 	(wire
 		(pts
+			(xy 81.28 179.07) (xy 81.28 167.64)
+		)
+		(stroke
+			(width 0)
+			(type default)
+		)
+	)
+	(wire
+		(pts
 			(xy 138.43 259.08) (xy 138.43 247.65)
 		)
@@
 		)
 	)
+	(wire
+		(pts
+			(xy 35.56 187.96) (xy 38.1 187.96)
+		)
+		(stroke
+			(width 0)
+			(type default)
+		)
+	)
 	(polyline
 		(pts
@@
 		)
 	)
+	(wire
+		(pts
+			(xy 19.05 190.5) (xy 31.75 190.5)
+		)
+		(stroke
+			(width 0)
+			(type default)
+		)
+	)
 	(polyline
 		(pts
@@
 		)
 	)
+	(label "VMA"
+		(at 59.69 190.5 0)
+		(effects
+			(font
+				(size 1.27 1.27)
+			)
+			(justify left bottom)
+		)
+	)
 	(label "RA7"
 		(at 173.99 162.56 0)
@@
 		)
 	)
+	(label "~{VMA}"
+		(at 26.67 190.5 0)
+		(effects
+			(font
+				(size 1.27 1.27)
+			)
+			(justify left bottom)
+		)
+	)
 	(label "RA0"
 		(at 163.83 144.78 0)
@@
 	)
 	(label "VMA"
-		(at 201.93 240.03 0)
+		(at 173.99 240.03 0)
 		(effects
 			(font
@@
 	(hierarchical_label "~{VMA}"
 		(shape input)
-		(at 107.95 167.64 180)
+		(at 19.05 190.5 180)
 		(effects
 			(font
@@
 		)
 	)
-	(hierarchical_label "VMA"
-		(shape input)
-		(at 160.02 240.03 180)
-		(effects
-			(font
-				(size 1.27 1.27)
-			)
-			(justify right)
-		)
-	)
 	(hierarchical_label "R~{W}B"
 		(shape input)
@@
 				)
 			)
+		)
+	)
+	(symbol
+		(lib_id "74xx:74LS02")
+		(at 45.72 190.5 0)
+		(unit 4)
+		(exclude_from_sim no)
+		(in_bom yes)
+		(on_board yes)
+		(dnp no)
+		(fields_autoplaced yes)
+		(property "Reference" "U7"
+			(at 45.72 181.61 0)
+			(effects
+				(font
+					(size 1.27 1.27)
+				)
+			)
+		)
+		(property "Value" "74LS02"
+			(at 45.72 184.15 0)
+			(effects
+				(font
+					(size 1.27 1.27)
+				)
+			)
+		)
+		(property "Footprint" ""
+			(at 45.72 190.5 0)
+			(effects
+				(font
+					(size 1.27 1.27)
+				)
+				(hide yes)
+			)
+		)
+		(property "Datasheet" "http://www.ti.com/lit/gpn/sn74ls02"
+			(at 45.72 190.5 0)
+			(effects
+				(font
+					(size 1.27 1.27)
+				)
+				(hide yes)
+			)
+		)
+		(property "Description" "quad 2-input NOR gate"
+			(at 45.72 190.5 0)
+			(effects
+				(font
+					(size 1.27 1.27)
+				)
+				(hide yes)
+			)
+		)
+		(pin "9"
+		)
+		(pin "4"
+		)
+		(pin "12"
+		)
+		(pin "13"
+		)
+		(pin "6"
+		)
+		(pin "10"
+		)
+		(pin "5"
+		)
+		(pin "1"
+		)
+		(pin "3"
+		)
+		(pin "2"
+		)
+		(pin "8"
+		)
+		(pin "7"
+		)
+		(pin "11"
+		)
+		(pin "14"
+		)
+		(instances
+			(project "Squale"
+				(path "/9e981419-a202-4dd8-b7ec-e1bde8e7b185/7d7f151b-a16e-4418-bf6d-71f4cdd2beb8"
+					(reference "U7")
+					(unit 4)
+				)
+			)

Commit message: WIP : passives parts, cosmetic stuffs.
Parts:
- added C17, C18, C19, C20, C21, C22, C23, C24, C25, C26, C27, C29, C30, C31, C36, C72: 100nF, symbol Device:C
- renumbered U2 to U24
Connections:
- net VCC5V: now also C17.1, C18.1, C19.1, C20.1, C21.1, C22.1, C23.1, C24.1, C25.1, C26.1, C27.1, C29.1, C30.1, C31.1, C36.1, C72.1
- net VSS: now also C17.2, C18.2, C19.2, C20.2, C21.2, C22.2, C23.2, C24.2, C25.2, C26.2, C27.2, C29.2, C30.2, C31.2, C36.2, C72.2
Other:
- moved on the sheet: U24C, U28G
