File: hardware/Motherboard/Squale.kicad_sch (KiCad schematic)
At the start: 0 parts

Commit message: wip
Other:
- sheet CPU ports: added SYS_ROM_BK, ~{VMA}; removed VMA
- sheet DRAM ports: added none; removed VMA
- sheet Sound ports: added LIGHTPEN_SWITCH; removed LIGHTPEN_INT
- sheet Video Controller ports: added LIGHTPEN_SWITCH; removed OpticalCK
Changed lines of the file:
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@@
 	)
 	(junction
-		(at 171.45 102.87)
+		(at 153.67 217.17)
 		(diameter 0)
 		(color 0 0 0 0)
 	)
 	(junction
-		(at 209.55 105.41)
+		(at 171.45 102.87)
 		(diameter 0)
 		(color 0 0 0 0)
 	)
 	(junction
-		(at 151.13 217.17)
+		(at 209.55 105.41)
 		(diameter 0)
 		(color 0 0 0 0)
@@
 	(wire
 		(pts
-			(xy 228.6 177.8) (xy 231.14 177.8)
+			(xy 228.6 177.8) (xy 233.68 177.8)
 		)
 		(stroke
@@
 	(wire
 		(pts
-			(xy 138.43 156.21) (xy 144.78 156.21)
+			(xy 138.43 156.21) (xy 148.59 156.21)
 		)
 		(stroke
@@
 	(wire
 		(pts
-			(xy 26.67 217.17) (xy 151.13 217.17)
+			(xy 22.86 217.17) (xy 153.67 217.17)
 		)
 		(stroke
@@
 	(wire
 		(pts
-			(xy 144.78 156.21) (xy 144.78 189.23)
+			(xy 148.59 156.21) (xy 148.59 189.23)
 		)
 		(stroke
@@
 	(wire
 		(pts
+			(xy 25.4 214.63) (xy 25.4 172.72)
+		)
+		(stroke
+			(width 0)
+			(type default)
+		)
+	)
+	(wire
+		(pts
 			(xy 48.26 110.49) (xy 102.87 110.49)
 		)
@@
 	(wire
 		(pts
+			(xy 142.24 214.63) (xy 25.4 214.63)
+		)
+		(stroke
+			(width 0)
+			(type default)
+		)
+	)
+	(wire
+		(pts
 			(xy 243.84 154.94) (xy 243.84 62.23)
 		)
@@
 		)
 	)
+	(wire
+		(pts
+			(xy 241.3 173.99) (xy 247.65 173.99)
+		)
+		(stroke
+			(width 0)
+			(type default)
+		)
+	)
+	(wire
+		(pts
+			(xy 241.3 199.39) (xy 241.3 173.99)
+		)
+		(stroke
+			(width 0)
+			(type default)
+		)
+	)
 	(bus
 		(pts
@@
 	(wire
 		(pts
-			(xy 26.67 217.17) (xy 26.67 168.91)
+			(xy 22.86 217.17) (xy 22.86 168.91)
 		)
 		(stroke
@@
 	(wire
 		(pts
-			(xy 144.78 189.23) (xy 316.23 189.23)
+			(xy 148.59 189.23) (xy 316.23 189.23)
 		)
 		(stroke
@@
 	(wire
 		(pts
-			(xy 147.32 153.67) (xy 147.32 186.69)
+			(xy 151.13 153.67) (xy 151.13 186.69)
+		)
+		(stroke
+			(width 0)
+			(type default)
+		)
+	)
+	(wire
+		(pts
+			(xy 403.86 193.04) (xy 406.4 193.04)
 		)
 		(stroke
@@
 	(wire
 		(pts
-			(xy 231.14 217.17) (xy 151.13 217.17)
+			(xy 233.68 217.17) (xy 153.67 217.17)
 		)
 		(stroke
@@
 	(wire
 		(pts
-			(xy 151.13 167.64) (xy 156.21 167.64)
+			(xy 153.67 167.64) (xy 156.21 167.64)
 		)
 		(stroke
@@
 	(wire
 		(pts
-			(xy 151.13 167.64) (xy 151.13 217.17)
+			(xy 153.67 167.64) (xy 153.67 217.17)
 		)
 		(stroke
@@
 		)
 	)
+	(wire
+		(pts
+			(xy 138.43 163.83) (xy 142.24 163.83)
+		)
+		(stroke
+			(width 0)
+			(type default)
+		)
+	)
 	(bus
 		(pts
@@
 	(wire
 		(pts
+			(xy 406.4 193.04) (xy 406.4 199.39)
+		)
+		(stroke
+			(width 0)
+			(type default)
+		)
+	)
+	(wire
+		(pts
 			(xy 22.86 69.85) (xy 38.1 69.85)
 		)
@@
 	(wire
 		(pts
-			(xy 231.14 177.8) (xy 231.14 217.17)
+			(xy 233.68 177.8) (xy 233.68 217.17)
 		)
 		(stroke
@@
 	(wire
 		(pts
-			(xy 138.43 158.75) (xy 142.24 158.75)
+			(xy 138.43 158.75) (xy 146.05 158.75)
 		)
 		(stroke
@@
 	(wire
 		(pts
-			(xy 142.24 158.75) (xy 142.24 191.77)
+			(xy 146.05 158.75) (xy 146.05 191.77)
 		)
 		(stroke
@@
 	(wire
 		(pts
-			(xy 142.24 191.77) (xy 318.77 191.77)
+			(xy 146.05 191.77) (xy 318.77 191.77)
 		)
 		(stroke
@@
 	(wire
 		(pts
+			(xy 25.4 172.72) (xy 30.48 172.72)
+		)
+		(stroke
+			(width 0)
+			(type default)
+		)
+	)
+	(wire
+		(pts
 			(xy 25.4 72.39) (xy 191.77 72.39)
 		)
@@
 	(wire
 		(pts
-			(xy 26.67 168.91) (xy 30.48 168.91)
+			(xy 22.86 168.91) (xy 30.48 168.91)
 		)
 		(stroke
@@
 	(wire
 		(pts
-			(xy 147.32 186.69) (xy 191.77 186.69)
+			(xy 406.4 199.39) (xy 241.3 199.39)
+		)
+		(stroke
+			(width 0)
+			(type default)
+		)
+	)
+	(wire
+		(pts
+			(xy 151.13 186.69) (xy 191.77 186.69)
 		)
 		(stroke
@@
 	(wire
 		(pts
-			(xy 138.43 153.67) (xy 147.32 153.67)
+			(xy 138.43 153.67) (xy 151.13 153.67)
 		)
 		(stroke
@@
 		)
 	)
+	(wire
+		(pts
+			(xy 142.24 163.83) (xy 142.24 214.63)
+		)
+		(stroke
+			(width 0)
+			(type default)
+		)
+	)
 	(bus
 		(pts
@@
 			)
 		)
-		(pin "VMA" output
-			(at 80.01 157.48 0)
-			(effects
-				(font
-					(size 1.27 1.27)
-				)
-				(justify right)
-			)
-		)
 		(pin "QB" output
 			(at 48.26 142.24 90)
@@
 			)
 		)
+		(pin "~{VMA}" output
+			(at 80.01 157.48 0)
+			(effects
+				(font
+					(size 1.27 1.27)
+				)
+				(justify right)
+			)
+		)
+		(pin "SYS_ROM_BK" input
+			(at 30.48 172.72 180)
+			(effects
+				(font
+					(size 1.27 1.27)
+				)
+				(justify left)
+			)
+		)
 		(instances
 			(project "Squale"
@@
 			)
 		)
-		(pin "OpticalCK" output
-			(at 368.3 185.42 180)
-			(effects
-				(font
-					(size 1.27 1.27)
-				)
-				(justify left)
-			)
-		)
 		(pin "~{CS_V1}" input
 			(at 398.78 142.24 90)
@@
 			)
 		)
+		(pin "LIGHTPEN_SWITCH" output
+			(at 403.86 193.04 0)
+			(effects
+				(font
+					(size 1.27 1.27)
+				)
+				(justify right)
+			)
+		)
 		(instances
 			(project "Squale"
@@
 		)
 		(pin "~{VMA}" input
-			(at 86.36 154.94 180)
-			(effects
-				(font
-					(size 1.27 1.27)
-				)
-				(justify left)
-			)
-		)
-		(pin "VMA" input
 			(at 86.36 157.48 180)
 			(effects
@@
 			)
 		)
-		(pin "LIGHTPEN_INT" input
-			(at 247.65 173.99 180)
-			(effects
-				(font
-					(size 1.27 1.27)
-				)
-				(justify left)
-			)
-		)
 		(pin "A0" input
 			(at 260.35 142.24 90)
@@
 			(effects
 				(font
+					(size 1.27 1.27)
+				)
+				(justify left)
+			)
+		)
+		(pin "LIGHTPEN_SWITCH" input
+			(at 247.65 173.99 180)
+			(effects
+				(font

Commit message: WIP : passives parts, cosmetic stuffs.
Other:
- removed sheet System Register
- sheet CPU ports: added SYS_COL[3..0], SYS_KEYB_LED, SYS_MDM_LINE, SYS_MDM_MC_~{BC}, ~{RSTB}; removed SYS_ROM_BK, ~{CS_REG}
