File: hardware/Motherboard/external_bus.kicad_sch (KiCad schematic)
At the start: 3 parts, among them J4 DB25_Socket, U30 74LS245, U31 74LS541

Commit message: WIP : passives parts, cosmetic stuffs.
Parts:
- added C37, C38: 100nF, symbol Device:C
Connections:
- net VCC5V: now also C37.1, C38.1
- net VSS: now also C37.2, C38.2
Other:
- moved on the sheet: J4, U30, U31

Commit message: Footprints.
Parts:
- C37, C38: footprint (none) -> Capacitor_THT:C_Disc_D9.0mm_W2.5mm_P5.00mm
- J4: footprint (none) -> Connector_Dsub:DSUB-25_Pins_Horizontal_P2.77x2.54mm_EdgePinOffset9.40mm
- U30, U31: footprint (none) -> Package_DIP:DIP-20_W7.62mm_Socket
Changed lines of the file:
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@@
 			)
 		)
-		(property "Footprint" ""
+		(property "Footprint" "Package_DIP:DIP-20_W7.62mm_Socket"
 			(at 224.79 175.26 0)
 			(effects
@@
 			)
 		)
-		(property "Footprint" ""
+		(property "Footprint" "Capacitor_THT:C_Disc_D9.0mm_W2.5mm_P5.00mm"
 			(at 240.9952 120.65 0)
 			(effects
@@
 			)
 		)
-		(property "Footprint" ""
+		(property "Footprint" "Package_DIP:DIP-20_W7.62mm_Socket"
 			(at 227.33 92.71 0)
 			(effects
@@
 			)
 		)
-		(property "Footprint" ""
+		(property "Footprint" "Connector_Dsub:DSUB-25_Pins_Horizontal_P2.77x2.54mm_EdgePinOffset9.40mm"
 			(at 300.99 128.27 0)
 			(effects
@@
 			)
 		)
-		(property "Footprint" ""
+		(property "Footprint" "Capacitor_THT:C_Disc_D9.0mm_W2.5mm_P5.00mm"
 			(at 206.7052 196.85 0)
 			(effects
