File: hardware/Motherboard/ROM_pack.kicad_sch (KiCad schematic)
At the start: 0 parts

Commit message: WIP
Other:
- title: (none) -> Apollo 7 Squale 
Changed lines of the file:
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@@
 	(generator_version "9.0")
 	(paper "A3")
+	(title_block
+		(title "Apollo 7 Squale ")
+		(rev "0.1")
+		(comment 1 "http://hxc2001.free.fr/Squale/")
+		(comment 2 "CC-BY Licence (Creative Commons Attribution)")
+		(comment 3 "Drawn by Jean-François DEL NERO")
+	)
 )

Commit message: WIP -rom pack
Parts:
- added J2: Conn_02x20_Odd_Even, symbol Connector_Generic_Shielded:Conn_02x20_Odd_Even_Shielded
- added J3: DA15_Socket, symbol Connector:DA15_Socket
- added U72: 6821, Package_DIP:DIP-40_W15.24mm, symbol Interface:6821
- added U73, U74: 74LS393, symbol 74xx:74LS393
Connections:
- new net: U72.39 (CA2), U73.1 (CP)
- new net EB: U72.25 (ENABLE)
- new net PA0: U72.36 (RS0)
- new net PA1: U72.35 (RS1)
- new net PA3: U72.24 (CS1)
- new net PD0: U72.33 (D0)
- new net PD1: U72.32 (D1)
- new net PD2: U72.31 (D2)
- new net PD3: U72.30 (D3)
- new net PD4: U72.29 (D4)
- new net PD5: U72.28 (D5)
- new net PD6: U72.27 (D6)
- new net PD7: U72.26 (D7)
- new net PRT_ACK: J3.5, U72.18 (CB1)
- new net PRT_D0: J3.15 (P15), U72.10 (PB0)
- new net PRT_D1: J3.14 (P14), U72.11 (PB1)
- new net PRT_D2: J3.13 (P13), U72.12 (PB2)
- new net PRT_D3: J3.12 (P12), U72.13 (PB3)
- new net PRT_D4: J3.11 (P111), U72.14 (PB4)
- new net PRT_D5: J3.10 (P10), U72.15 (PB5)
- new net PRT_D6: J3.9 (P9), U72.16 (PB6)
- new net PRT_D7: J3.4, U72.17 (PB7)
- new net PRT_STROBE: J3.6, U72.19 (CB2)
- new net ROMPACK_RST_ADDR: U73.12 (MR), U73.2 (MR), U74.12 (MR), U74.2 (MR)
- new net RP_A0: J2.6 (Pin_6), U73.3 (Q0)
- new net RP_A1: J2.8 (Pin_8), U73.4 (Q1)
- new net RP_A10: J2.26 (Pin_26), U74.5 (Q2)
- new net RP_A11: J2.28 (Pin_28), U74.13 (CP), U74.6 (Q3)
- new net RP_A12: J2.30 (Pin_30), U74.11 (Q0)
- new net RP_A13: J2.32 (Pin_32), U74.10 (Q1)
- new net RP_A14: J2.34 (Pin_34), U74.9 (Q2)
- new net RP_A15: J2.36 (Pin_36), U74.8 (Q3)
- new net RP_A2: J2.10 (Pin_10), U73.5 (Q2)
- new net RP_A3: J2.12 (Pin_12), U73.13 (CP), U73.6 (Q3)
- new net RP_A4: J2.14 (Pin_14), U73.11 (Q0)
- new net RP_A5: J2.16 (Pin_16), U73.10 (Q1)
- new net RP_A6: J2.18 (Pin_18), U73.9 (Q2)
- new net RP_A7: J2.20 (Pin_20), U73.8 (Q3), U74.1 (CP)
- new net RP_A8: J2.22 (Pin_22), U74.3 (Q0)
- new net RP_A9: J2.24 (Pin_24), U74.4 (Q1)
- new net RP_D0: J2.5 (Pin_5), U72.2 (PA0)
- new net RP_D1: J2.7 (Pin_7), U72.3 (PA1)
- new net RP_D2: J2.9 (Pin_9), U72.4 (PA2)
- new net RP_D3: J2.11 (Pin_11), U72.5 (PA3)
- new net RP_D4: J2.13 (Pin_13), U72.6 (PA4)
- new net RP_D5: J2.15 (Pin_15), U72.7 (PA5)
- new net RP_D6: J2.17 (Pin_17), U72.8 (PA6)
- new net RP_D7: J2.19 (Pin_19), U72.9 (PA7)
- new net R~{W}B: U72.21 (R/~{W})
- new net VCC5V: J2.37 (Pin_37), J2.38 (Pin_38), J2.39 (Pin_39), J2.40 (Pin_40), U72.20 (VCC), U72.22 (CS0), U73.14 (VCC), U74.14 (VCC)
- new net VSS: J2.1 (Pin_1), J2.2 (Pin_2), J2.3 (Pin_3), J2.4 (Pin_4), J3.2, J3.3, U72.1 (VSS), U73.7 (GND), U74.7 (GND)
- new net ~{CS_PIA}: U72.23 (~{CS2})
- new net ~{RSTB}: U72.34 (~{RESET})
- no-connect marks 0 -> 14
Other:
- note added: "Base : 0xF048"
- title: Apollo 7 Squale  -> Apollo 7 Squale - ROMPack and Printer ports

Commit message: wip
Other:
- moved on the sheet: U74C
Changed lines of the file:
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@@
 	(symbol
 		(lib_id "power:VSS")
-		(at 393.7 219.71 0)
+		(at 378.46 220.98 0)
 		(unit 1)
 		(exclude_from_sim no)
@@
 		(fields_autoplaced yes)
 		(property "Reference" "#PWR0229"
-			(at 393.7 223.52 0)
+			(at 378.46 224.79 0)
 			(effects
 				(font
@@
 		)
 		(property "Value" "VCC5V"
-			(at 393.7 214.63 0)
-			(effects
-				(font
-					(size 1.27 1.27)
-				)
-			)
-		)
-		(property "Footprint" ""
-			(at 393.7 219.71 0)
+			(at 378.46 215.9 0)
+			(effects
+				(font
+					(size 1.27 1.27)
+				)
+			)
+		)
+		(property "Footprint" ""
+			(at 378.46 220.98 0)
 			(effects
 				(font
@@
 		)
 		(property "Datasheet" ""
-			(at 393.7 219.71 0)
+			(at 378.46 220.98 0)
 			(effects
 				(font
@@
 		)
 		(property "Description" "Power symbol creates a global label with name \"VSS\""
-			(at 393.7 219.71 0)
+			(at 378.46 220.98 0)
 			(effects
 				(font
@@
 	(symbol
 		(lib_id "74xx:74LS393")
-		(at 393.7 232.41 0)
+		(at 378.46 233.68 0)
 		(unit 3)
 		(exclude_from_sim no)
@@
 		(fields_autoplaced yes)
 		(property "Reference" "U74"
-			(at 400.05 231.1399 0)
+			(at 384.81 232.4099 0)
 			(effects
 				(font
@@
 		)
 		(property "Value" "74LS393"
-			(at 400.05 233.6799 0)
+			(at 384.81 234.9499 0)
 			(effects
 				(font
@@
 		)
 		(property "Footprint" ""
-			(at 393.7 232.41 0)
+			(at 378.46 233.68 0)
 			(effects
 				(font
@@
 		)
 		(property "Datasheet" "74xx\\74LS393.pdf"
-			(at 393.7 232.41 0)
+			(at 378.46 233.68 0)
 			(effects
 				(font
@@
 		)
 		(property "Description" "Dual BCD 4-bit counter"
-			(at 393.7 232.41 0)
+			(at 378.46 233.68 0)
 			(effects
 				(font
@@
 	(symbol
 		(lib_id "power:GND")
-		(at 393.7 245.11 0)
+		(at 378.46 246.38 0)
 		(unit 1)
 		(exclude_from_sim no)
@@
 		(fields_autoplaced yes)
 		(property "Reference" "#PWR0227"
-			(at 393.7 251.46 0)
+			(at 378.46 252.73 0)
 			(effects
 				(font
@@
 		)
 		(property "Value" "VSS"
-			(at 393.7 250.19 0)
-			(effects
-				(font
-					(size 1.27 1.27)
-				)
-				(hide yes)
-			)
-		)
-		(property "Footprint" ""
-			(at 393.7 245.11 0)
+			(at 378.46 251.46 0)
+			(effects
+				(font
+					(size 1.27 1.27)
+				)
+				(hide yes)
+			)
+		)
+		(property "Footprint" ""
+			(at 378.46 246.38 0)
 			(effects
 				(font
@@
 		)
 		(property "Datasheet" ""
-			(at 393.7 245.11 0)
+			(at 378.46 246.38 0)
 			(effects
 				(font
@@
 		)
 		(property "Description" "Power symbol creates a global label with name \"GND\" , ground"
-			(at 393.7 245.11 0)
-			(effects
-				(font
+			(at 378.46 246.38 0)
+			(effects
+				(font

Commit message: WIP : passives parts, cosmetic stuffs.
Parts:
- added C34, C70: 100nF, symbol Device:C
Connections:
- net VCC5V: now also C34.1, C70.1
- net VSS: now also C34.2, C70.2

Commit message: Footprints.
Parts:
- C34, C70: footprint (none) -> Capacitor_THT:C_Disc_D9.0mm_W2.5mm_P5.00mm
- J2: footprint (none) -> Connector_PinSocket_2.54mm:PinSocket_2x20_P2.54mm_Vertical
- J3: footprint (none) -> Connector_Dsub:DSUB-15_Socket_Horizontal_P2.77x2.84mm_EdgePinOffset9.40mm
- U72: footprint Package_DIP:DIP-40_W15.24mm -> Package_DIP:DIP-40_W15.24mm_Socket
- U73, U74: footprint (none) -> Package_DIP:DIP-14_W7.62mm_Socket
Changed lines of the file:
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@@
 			)
 		)
-		(property "Footprint" "Package_DIP:DIP-40_W15.24mm"
+		(property "Footprint" "Package_DIP:DIP-40_W15.24mm_Socket"
 			(at 209.55 123.19 0)
 			(effects
@@
 			)
 		)
-		(property "Footprint" ""
+		(property "Footprint" "Connector_Dsub:DSUB-15_Socket_Horizontal_P2.77x2.84mm_EdgePinOffset9.40mm"
 			(at 331.47 191.77 0)
 			(effects
@@
 			)
 		)
-		(property "Footprint" ""
+		(property "Footprint" "Package_DIP:DIP-14_W7.62mm_Socket"
 			(at 269.24 96.52 0)
 			(effects
@@
 			)
 		)
-		(property "Footprint" ""
+		(property "Footprint" "Connector_PinSocket_2.54mm:PinSocket_2x20_P2.54mm_Vertical"
 			(at 327.66 76.2 0)
 			(effects
@@
 			)
 		)
-		(property "Footprint" ""
+		(property "Footprint" "Package_DIP:DIP-14_W7.62mm_Socket"
 			(at 269.24 143.51 0)
 			(effects
@@
 			)
 		)
-		(property "Footprint" ""
+		(property "Footprint" "Package_DIP:DIP-14_W7.62mm_Socket"
 			(at 378.46 233.68 0)
 			(effects
@@
 			)
 		)
-		(property "Footprint" ""
+		(property "Footprint" "Package_DIP:DIP-14_W7.62mm_Socket"
 			(at 269.24 120.65 0)
 			(effects
@@
 			)
 		)
-		(property "Footprint" ""
+		(property "Footprint" "Capacitor_THT:C_Disc_D9.0mm_W2.5mm_P5.00mm"
 			(at 301.9552 143.51 0)
 			(effects
@@
 			)
 		)
-		(property "Footprint" ""
+		(property "Footprint" "Capacitor_THT:C_Disc_D9.0mm_W2.5mm_P5.00mm"
 			(at 192.7352 44.45 0)
 			(effects
@@
 			)
 		)
-		(property "Footprint" ""
+		(property "Footprint" "Package_DIP:DIP-14_W7.62mm_Socket"
 			(at 269.24 71.12 0)
 			(effects
@@
 			)
 		)
-		(property "Footprint" ""
+		(property "Footprint" "Package_DIP:DIP-14_W7.62mm_Socket"
 			(at 353.06 233.68 0)
 			(effects

Commit message: fix footprint
Parts:
- J3: footprint Connector_Dsub:DSUB-15_Socket_Horizontal_P2.77x2.84mm_EdgePinOffset9.40mm -> Connector_Dsub:DSUB-15_Pins_Horizontal_P2.77x2.84mm_EdgePinOffset9.40mm
Changed lines of the file:
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@@
 			)
 		)
-		(property "Footprint" "Connector_Dsub:DSUB-15_Socket_Horizontal_P2.77x2.84mm_EdgePinOffset9.40mm"
+		(property "Footprint" "Connector_Dsub:DSUB-15_Pins_Horizontal_P2.77x2.84mm_EdgePinOffset9.40mm"
 			(at 331.47 191.77 0)
 			(effects

Commit message: Connectors footprint.
Parts:
- J2: footprint Connector_PinSocket_2.54mm:PinSocket_2x20_P2.54mm_Vertical -> Library:Ribbon_Conn
Changed lines of the file:
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@@
 			)
 		)
-		(property "Footprint" "Connector_PinSocket_2.54mm:PinSocket_2x20_P2.54mm_Vertical"
+		(property "Footprint" "Library:Ribbon_Conn"
 			(at 327.66 76.2 0)
 			(effects
