File: hardware/Motherboard/Squale.kicad_pcb (KiCad board)
At the start: 2 copper layers, 218 parts, among them J10 DA15_Socket, J11 Conn_01x22_Socket, J2 Conn_02x20_Odd_Even, J3 DA15_Socket, J4 DB25_Socket, J5 DIN-5_180degree, J6 DE9_Socket, J7 DE9_Pins, J8 DE9_Pins, J9 DIN-5_180degree, P1 VR10K, Q1 2N2222, Q2 2N2222, Q3 2N2222, Q4 2N2222, Q5 2N2222, Q6 2N2222, Q7 2N2222, U1 MC6809, U10 74LS138, U11 74LS245, U12 74LS541, U13 74LS541, U14 74LS541, U15 74LS393, U16 MK4164N, U17 MK4164N, U18 MK4164N, U19 MK4164N, U2 27C64, U20 MK4164N, U21 MK4164N, U22 MK4164N, U23 MK4164N, U24 74LS123, U25 74LS74, U26 74LS74, U28 74LS04, U29 74LS02, U3 74LS245, U30 74LS245, U31 74LS541, U32 74LS04, U33 74LS17, U34 74LS166, U35 74LS166, U36 74LS166, U37 74LS166, U38 MK4116N, U39 MK4116N, U4 74LS139, U40 MK4116N, U41 MK4116N, U42 MK4116N, U43 MK4116N, U44 MK4116N, U45 MK4116N, U46 MK4116N, U47 MK4116N, U48 MK4116N, U49 MK4116N, U5 74LS20, U50 MK4116N, U51 MK4116N, U52 MK4116N, U53 MK4116N, U54 74LS374, U55 74LS374, U56 74LS541, U57 74LS32, U58 74LS374, U59 EF9365, U6 74LS08, U60 74LS04, U61 74LS193, U62 TBP18S030N, U63 74LS32, U64 74LS374, U65 AY-3-8910A, U66 74LS273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

Commit message: first ICs approximate placement
Parts:
- moved U15 445.2 mm to (526.6, 269.5)
- moved U23 429.9 mm to (534.2, 310.3), turned to 180 degrees
- moved U22 429.3 mm to (521.6, 310.3), turned to 180 degrees
- moved U21 428.7 mm to (509.1, 310.3), turned to 180 degrees
- moved U20 428.2 mm to (496.6, 310.3), turned to 180 degrees
- moved U19 427.9 mm to (484.4, 310.3), turned to 180 degrees
- moved U18 427.1 mm to (471.6, 310.3), turned to 180 degrees
- moved U17 426.6 mm to (459.1, 310.2), turned to 180 degrees
- moved U16 426.0 mm to (446.6, 310.2), turned to 180 degrees
- moved U1 403.9 mm to (478.4, 226.6)
- moved U11 392.1 mm to (461.8, 286.7), turned to 90 degrees
- moved U14 390.5 mm to (514.0, 261.8)
- moved U13 389.9 mm to (501.5, 261.8)
- moved U2 386.1 mm to (472.6, 267.3), turned to 180 degrees
- moved U12 383.9 mm to (501.6, 232.6)
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
Commit message: Full & scripted placement, based on the PCBAnnot data.
Parts:
- J3: moved to B.Cu
- moved C14 342.5 mm to (148.3, 149.7), turned to 90 degrees
- moved C15 339.5 mm to (160.8, 148.3), turned to -90 degrees
- moved R49 329.8 mm to (107.3, 258.3), turned to -90 degrees
- moved R40 318.2 mm to (152.1, 144.7), turned to -90 degrees
- moved R39 315.8 mm to (156.1, 144.7), turned to -90 degrees
- moved R19 313.2 mm to (84.6, 260.8), turned to -90 degrees
- moved R17 310.3 mm to (93.6, 255.9), turned to -90 degrees
- moved R38 307.8 mm to (166.0, 144.6), turned to -90 degrees
- moved R18 307.7 mm to (97.6, 260.7), turned to -90 degrees
- moved R42 289.3 mm to (500.8, 211.8), turned to -90 degrees
- moved R23 284.0 mm to (360.3, 178.9), turned to -90 degrees
- moved C62 269.9 mm to (125.5, 277.1)
- moved R24 266.8 mm to (352.7, 163.5), turned to -90 degrees
- moved C19 261.0 mm to (515.7, 284.9), turned to 180 degrees
- moved R27 259.5 mm to (360.6, 147.2), turned to -90 degrees
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
Commit message: Fix DRAM address bus connection.
Parts:
- U24: footprint Package_DIP:DIP-14_W7.62mm_Socket -> Package_DIP:DIP-16_W7.62mm_Socket
- moved P1 6.24 mm to (349.5, 216.0), turned to 90 degrees
Connections:
- U16 pad 10: unconnected-(U16-A5-Pad10) -> /DRAM/RA5
- U16 pad 11: unconnected-(U16-A4-Pad11) -> /DRAM/RA4
- U16 pad 12: unconnected-(U16-A3-Pad12) -> /DRAM/RA3
- U16 pad 13: unconnected-(U16-A6-Pad13) -> /DRAM/RA6
- U16 pad 5: unconnected-(U16-A0-Pad5) -> /DRAM/RA0
- U16 pad 6: unconnected-(U16-A2-Pad6) -> /DRAM/RA2
- U16 pad 7: unconnected-(U16-A1-Pad7) -> /DRAM/RA1
- U16 pad 9: unconnected-(U16-A7-Pad9) -> /DRAM/RA7
- U17 pad 10: unconnected-(U17-A5-Pad10) -> /DRAM/RA5
- U17 pad 11: unconnected-(U17-A4-Pad11) -> /DRAM/RA4
- U17 pad 12: unconnected-(U17-A3-Pad12) -> /DRAM/RA3
- U17 pad 13: unconnected-(U17-A6-Pad13) -> /DRAM/RA6
- U17 pad 5: unconnected-(U17-A0-Pad5) -> /DRAM/RA0
- U17 pad 6: unconnected-(U17-A2-Pad6) -> /DRAM/RA2
- U17 pad 7: unconnected-(U17-A1-Pad7) -> /DRAM/RA1
- U17 pad 9: unconnected-(U17-A7-Pad9) -> /DRAM/RA7
- U18 pad 10: unconnected-(U18-A5-Pad10) -> /DRAM/RA5
- U18 pad 11: unconnected-(U18-A4-Pad11) -> /DRAM/RA4
- U18 pad 12: unconnected-(U18-A3-Pad12) -> /DRAM/RA3
- U18 pad 13: unconnected-(U18-A6-Pad13) -> /DRAM/RA6
- U18 pad 5: unconnected-(U18-A0-Pad5) -> /DRAM/RA0
- U18 pad 6: unconnected-(U18-A2-Pad6) -> /DRAM/RA2
- U18 pad 7: unconnected-(U18-A1-Pad7) -> /DRAM/RA1
- U18 pad 9: unconnected-(U18-A7-Pad9) -> /DRAM/RA7
- U19 pad 10: unconnected-(U19-A5-Pad10) -> /DRAM/RA5
- U19 pad 11: unconnected-(U19-A4-Pad11) -> /DRAM/RA4
- U19 pad 12: unconnected-(U19-A3-Pad12) -> /DRAM/RA3
- U19 pad 13: unconnected-(U19-A6-Pad13) -> /DRAM/RA6
- U19 pad 5: unconnected-(U19-A0-Pad5) -> /DRAM/RA0
- U19 pad 6: unconnected-(U19-A2-Pad6) -> /DRAM/RA2
- U19 pad 7: unconnected-(U19-A1-Pad7) -> /DRAM/RA1
- U19 pad 9: unconnected-(U19-A7-Pad9) -> /DRAM/RA7
- U20 pad 10: unconnected-(U20-A5-Pad10) -> /DRAM/RA5
- U20 pad 11: unconnected-(U20-A4-Pad11) -> /DRAM/RA4
- U20 pad 12: unconnected-(U20-A3-Pad12) -> /DRAM/RA3
- U20 pad 13: unconnected-(U20-A6-Pad13) -> /DRAM/RA6
- U20 pad 5: unconnected-(U20-A0-Pad5) -> /DRAM/RA0
- U20 pad 6: unconnected-(U20-A2-Pad6) -> /DRAM/RA2
- U20 pad 7: unconnected-(U20-A1-Pad7) -> /DRAM/RA1
- U20 pad 9: unconnected-(U20-A7-Pad9) -> /DRAM/RA7
- U21 pad 10: unconnected-(U21-A5-Pad10) -> /DRAM/RA5
- U21 pad 11: unconnected-(U21-A4-Pad11) -> /DRAM/RA4
- U21 pad 12: unconnected-(U21-A3-Pad12) -> /DRAM/RA3
- U21 pad 13: unconnected-(U21-A6-Pad13) -> /DRAM/RA6
- U21 pad 5: unconnected-(U21-A0-Pad5) -> /DRAM/RA0
- U21 pad 6: unconnected-(U21-A2-Pad6) -> /DRAM/RA2
- U21 pad 7: unconnected-(U21-A1-Pad7) -> /DRAM/RA1
- U21 pad 9: unconnected-(U21-A7-Pad9) -> /DRAM/RA7
- U22 pad 10: unconnected-(U22-A5-Pad10) -> /DRAM/RA5
- U22 pad 11: unconnected-(U22-A4-Pad11) -> /DRAM/RA4
- U22 pad 12: unconnected-(U22-A3-Pad12) -> /DRAM/RA3
- U22 pad 13: unconnected-(U22-A6-Pad13) -> /DRAM/RA6
- U22 pad 5: unconnected-(U22-A0-Pad5) -> /DRAM/RA0
- U22 pad 6: unconnected-(U22-A2-Pad6) -> /DRAM/RA2
- U22 pad 7: unconnected-(U22-A1-Pad7) -> /DRAM/RA1
- U22 pad 9: unconnected-(U22-A7-Pad9) -> /DRAM/RA7
- U23 pad 10: unconnected-(U23-A5-Pad10) -> /DRAM/RA5
- U23 pad 11: unconnected-(U23-A4-Pad11) -> /DRAM/RA4
- U23 pad 12: unconnected-(U23-A3-Pad12) -> /DRAM/RA3
- U23 pad 13: unconnected-(U23-A6-Pad13) -> /DRAM/RA6
- U23 pad 5: unconnected-(U23-A0-Pad5) -> /DRAM/RA0
- U23 pad 6: unconnected-(U23-A2-Pad6) -> /DRAM/RA2
- U23 pad 7: unconnected-(U23-A1-Pad7) -> /DRAM/RA1
- U23 pad 9: unconnected-(U23-A7-Pad9) -> /DRAM/RA7

Commit message: WIP : Motherboard layout.
Parts:
- U2: value 27C64 -> 27C32; footprint Package_DIP:DIP-28_W15.24mm_Socket -> Package_DIP:DIP-24_18.0mmx34.29mm_W15.24mm
- moved R28 12.9 mm to (316.7, 160.0), turned to 90 degrees
- moved R35 12.9 mm to (337.1, 160.0), turned to 90 degrees
- moved R45 12.9 mm to (486.4, 200.7), turned to 90 degrees
- moved R43 12.9 mm to (482.6, 200.7), turned to 90 degrees
- moved R44 12.9 mm to (478.8, 200.7), turned to 90 degrees
- moved R21 12.8 mm to (286.3, 238.3), turned to 90 degrees
- moved R47 12.8 mm to (328.2, 160.0), turned to 90 degrees
- moved R36 12.8 mm to (340.9, 160.0), turned to 90 degrees
- moved R37 12.8 mm to (333.2, 160.0), turned to 90 degrees
- moved R29 12.7 mm to (344.7, 160.0), turned to 90 degrees
- moved R42 12.7 mm to (500.4, 224.5), turned to 90 degrees
- moved R26 12.7 mm to (356.1, 159.8), turned to 90 degrees
- moved R23 12.7 mm to (359.9, 191.5), turned to 90 degrees
- moved R38 12.6 mm to (166.1, 157.2), turned to 90 degrees
- moved R33 12.5 mm to (320.5, 160.0), turned to 90 degrees
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Connections:
- P1 pad 1: Net-(U68-VREF) -> VSS
- P1 pad 3: VSS -> Net-(U68-VREF)
- U10 pad 4: VCC5V -> VSS
- U10 pad 6: unconnected-(U10-E3-Pad6) -> /CPU/EB
- U16 pad 11: /DRAM/RA4 -> /DRAM/RA3
- U16 pad 12: /DRAM/RA3 -> /DRAM/RA1
- U16 pad 13: /DRAM/RA6 -> /DRAM/RA0
- U16 pad 5: /DRAM/RA0 -> /DRAM/RA2
- U16 pad 6: /DRAM/RA2 -> /DRAM/RA4
- U16 pad 7: /DRAM/RA1 -> /DRAM/RA6
- U17 pad 11: /DRAM/RA4 -> /DRAM/RA3
- U17 pad 12: /DRAM/RA3 -> /DRAM/RA1
- U17 pad 13: /DRAM/RA6 -> /DRAM/RA0
- U17 pad 5: /DRAM/RA0 -> /DRAM/RA2
- U17 pad 6: /DRAM/RA2 -> /DRAM/RA4
- U17 pad 7: /DRAM/RA1 -> /DRAM/RA6
- U18 pad 11: /DRAM/RA4 -> /DRAM/RA3
- U18 pad 12: /DRAM/RA3 -> /DRAM/RA1
- U18 pad 13: /DRAM/RA6 -> /DRAM/RA0
- U18 pad 5: /DRAM/RA0 -> /DRAM/RA2
- U18 pad 6: /DRAM/RA2 -> /DRAM/RA4
- U18 pad 7: /DRAM/RA1 -> /DRAM/RA6
- U19 pad 11: /DRAM/RA4 -> /DRAM/RA3
- U19 pad 12: /DRAM/RA3 -> /DRAM/RA1
- U19 pad 13: /DRAM/RA6 -> /DRAM/RA0
- U19 pad 5: /DRAM/RA0 -> /DRAM/RA2
- U19 pad 6: /DRAM/RA2 -> /DRAM/RA4
- U19 pad 7: /DRAM/RA1 -> /DRAM/RA6
- U2 pad 1: unconnected-(U2-VPP-Pad1) -> /A7
- U2 pad 10: /A0 -> /D1
- U2 pad 11: /D0 -> /D2
- U2 pad 12: /D1 -> VSS
- U2 pad 13: /D2 -> /D3
- U2 pad 14: VSS -> /D4
- U2 pad 15: /D3 -> /D5
- U2 pad 16: /D4 -> /D6
- U2 pad 17: /D5 -> /D7
- U2 pad 18: /D6 -> /CPU/~{CSROM}
- U2 pad 19: /D7 -> /A10
- U2 pad 2: /CPU/SYS_ROM_BK -> /A6
- U2 pad 21: /A10 -> /A11
- U2 pad 22: unconnected-(U2-~{OE}-Pad22) -> /A9
- U2 pad 23: /A11 -> /A8
- U2 pad 24: /A9 -> unconnected-(U2-VCC-Pad24)
- U2 pad 3: /A7 -> /A5
- U2 pad 4: /A6 -> /A4
- U2 pad 5: /A5 -> /A3
- U2 pad 6: /A4 -> /A2
- U2 pad 7: /A3 -> /A1
- U2 pad 8: /A2 -> /A0
- U2 pad 9: /A1 -> /D0
- U20 pad 11: /DRAM/RA4 -> /DRAM/RA3
- U20 pad 12: /DRAM/RA3 -> /DRAM/RA1
- U20 pad 13: /DRAM/RA6 -> /DRAM/RA0
- U20 pad 5: /DRAM/RA0 -> /DRAM/RA2
- U20 pad 6: /DRAM/RA2 -> /DRAM/RA4
- U20 pad 7: /DRAM/RA1 -> /DRAM/RA6
- U21 pad 11: /DRAM/RA4 -> /DRAM/RA3
- U21 pad 12: /DRAM/RA3 -> /DRAM/RA1
- U21 pad 13: /DRAM/RA6 -> /DRAM/RA0
- U21 pad 5: /DRAM/RA0 -> /DRAM/RA2
- U21 pad 6: /DRAM/RA2 -> /DRAM/RA4
- U21 pad 7: /DRAM/RA1 -> /DRAM/RA6
- U22 pad 11: /DRAM/RA4 -> /DRAM/RA3
- U22 pad 12: /DRAM/RA3 -> /DRAM/RA1
- U22 pad 13: /DRAM/RA6 -> /DRAM/RA0
- U22 pad 5: /DRAM/RA0 -> /DRAM/RA2
- U22 pad 6: /DRAM/RA2 -> /DRAM/RA4
- U22 pad 7: /DRAM/RA1 -> /DRAM/RA6
- U23 pad 11: /DRAM/RA4 -> /DRAM/RA3
- U23 pad 12: /DRAM/RA3 -> /DRAM/RA1
- U23 pad 13: /DRAM/RA6 -> /DRAM/RA0
- U23 pad 5: /DRAM/RA0 -> /DRAM/RA2
- U23 pad 6: /DRAM/RA2 -> /DRAM/RA4
- U23 pad 7: /DRAM/RA1 -> /DRAM/RA6
- U29 pad 6: /Sound/A0 -> /A0
- U3 pad 11: /PD7 -> /D7
- U3 pad 12: /PD6 -> /D6
- U3 pad 13: /PD5 -> /D5
- U3 pad 14: /PD4 -> /D4
- U3 pad 15: /PD3 -> /D3
- U3 pad 16: /PD2 -> /D2
- U3 pad 17: /PD1 -> /D1
- U3 pad 18: /PD0 -> /D0
- U3 pad 2: /D0 -> /PD0
- U3 pad 3: /D1 -> /PD1
- U3 pad 4: /D2 -> /PD2
- U3 pad 5: /D3 -> /PD3
- U3 pad 6: /D4 -> /PD4
- U3 pad 7: /D5 -> /PD5
- U3 pad 8: /D6 -> /PD6
- U3 pad 9: /D7 -> /PD7
- U34 pad 10: unconnected-(U34-E-Pad10) -> /Video Controller/~{D_{3}I}
- U34 pad 11: unconnected-(U34-F-Pad11) -> /Video Controller/~{D_{2}I}
- U34 pad 12: unconnected-(U34-G-Pad12) -> /Video Controller/~{D_{1}I}
- U34 pad 14: unconnected-(U34-H-Pad14) -> /Video Controller/~{D_{0}I}
- U35 pad 10: unconnected-(U35-E-Pad10) -> /Video Controller/~{D_{3}R}
- U35 pad 11: unconnected-(U35-F-Pad11) -> /Video Controller/~{D_{2}R}
- U35 pad 12: unconnected-(U35-G-Pad12) -> /Video Controller/~{D_{1}R}
- U35 pad 14: unconnected-(U35-H-Pad14) -> /Video Controller/~{D_{0}R}
- U36 pad 10: unconnected-(U36-E-Pad10) -> /Video Controller/~{D_{3}V}
- U36 pad 11: unconnected-(U36-F-Pad11) -> /Video Controller/~{D_{2}V}
- U36 pad 12: unconnected-(U36-G-Pad12) -> /Video Controller/~{D_{1}V}
- U36 pad 14: unconnected-(U36-H-Pad14) -> /Video Controller/~{D_{0}V}
- U37 pad 10: unconnected-(U37-E-Pad10) -> /Video Controller/~{D_{3}B}
- U37 pad 11: unconnected-(U37-F-Pad11) -> /Video Controller/~{D_{2}B}
- U37 pad 12: unconnected-(U37-G-Pad12) -> /Video Controller/~{D_{1}B}
- U37 pad 14: unconnected-(U37-H-Pad14) -> /Video Controller/~{D_{0}B}
- U38 pad 10: /Video Controller/VA5 -> /Video Controller/VA0
- U38 pad 11: /Video Controller/VA4 -> /Video Controller/VA2
- U38 pad 12: /Video Controller/VA3 -> /Video Controller/VA4
- U38 pad 5: /Video Controller/VA0 -> /Video Controller/VA5
- U38 pad 6: /Video Controller/VA2 -> /Video Controller/VA3
- U39 pad 10: /Video Controller/VA5 -> /Video Controller/VA0
- U39 pad 11: /Video Controller/VA4 -> /Video Controller/VA2
- U39 pad 12: /Video Controller/VA3 -> /Video Controller/VA4
- U39 pad 5: /Video Controller/VA0 -> /Video Controller/VA5
- U39 pad 6: /Video Controller/VA2 -> /Video Controller/VA3
- U40 pad 10: /Video Controller/VA5 -> /Video Controller/VA0
- U40 pad 11: /Video Controller/VA4 -> /Video Controller/VA2
- U40 pad 12: /Video Controller/VA3 -> /Video Controller/VA4
- U40 pad 5: /Video Controller/VA0 -> /Video Controller/VA5
- U40 pad 6: /Video Controller/VA2 -> /Video Controller/VA3
- U41 pad 10: /Video Controller/VA5 -> /Video Controller/VA0
- U41 pad 11: /Video Controller/VA4 -> /Video Controller/VA2
- U41 pad 12: /Video Controller/VA3 -> /Video Controller/VA4
- U41 pad 5: /Video Controller/VA0 -> /Video Controller/VA5
- U41 pad 6: /Video Controller/VA2 -> /Video Controller/VA3
- U42 pad 10: /Video Controller/VA5 -> /Video Controller/VA0
- U42 pad 11: /Video Controller/VA4 -> /Video Controller/VA2
- U42 pad 12: /Video Controller/VA3 -> /Video Controller/VA4
- U42 pad 5: /Video Controller/VA0 -> /Video Controller/VA5
- U42 pad 6: /Video Controller/VA2 -> /Video Controller/VA3
- U43 pad 10: /Video Controller/VA5 -> /Video Controller/VA0
- U43 pad 11: /Video Controller/VA4 -> /Video Controller/VA2
- U43 pad 12: /Video Controller/VA3 -> /Video Controller/VA4
- U43 pad 5: /Video Controller/VA0 -> /Video Controller/VA5
- U43 pad 6: /Video Controller/VA2 -> /Video Controller/VA3
- U44 pad 10: /Video Controller/VA5 -> /Video Controller/VA0
- U44 pad 11: /Video Controller/VA4 -> /Video Controller/VA2
- U44 pad 12: /Video Controller/VA3 -> /Video Controller/VA4
- U44 pad 5: /Video Controller/VA0 -> /Video Controller/VA5
- U44 pad 6: /Video Controller/VA2 -> /Video Controller/VA3
- U45 pad 10: /Video Controller/VA5 -> /Video Controller/VA0
- U45 pad 11: /Video Controller/VA4 -> /Video Controller/VA2
- U45 pad 12: /Video Controller/VA3 -> /Video Controller/VA4
- U45 pad 5: /Video Controller/VA0 -> /Video Controller/VA5
- U45 pad 6: /Video Controller/VA2 -> /Video Controller/VA3
- U46 pad 10: /Video Controller/VA5 -> /Video Controller/VA0
- U46 pad 11: /Video Controller/VA4 -> /Video Controller/VA2
- U46 pad 12: /Video Controller/VA3 -> /Video Controller/VA4
- U46 pad 5: /Video Controller/VA0 -> /Video Controller/VA5
- U46 pad 6: /Video Controller/VA2 -> /Video Controller/VA3
- U47 pad 10: /Video Controller/VA5 -> /Video Controller/VA0
- U47 pad 11: /Video Controller/VA4 -> /Video Controller/VA2
- U47 pad 12: /Video Controller/VA3 -> /Video Controller/VA4
- U47 pad 5: /Video Controller/VA0 -> /Video Controller/VA5
- U47 pad 6: /Video Controller/VA2 -> /Video Controller/VA3
- U48 pad 10: /Video Controller/VA5 -> /Video Controller/VA0
- U48 pad 11: /Video Controller/VA4 -> /Video Controller/VA2
- U48 pad 12: /Video Controller/VA3 -> /Video Controller/VA4
- U48 pad 5: /Video Controller/VA0 -> /Video Controller/VA5
- U48 pad 6: /Video Controller/VA2 -> /Video Controller/VA3
- U49 pad 10: /Video Controller/VA5 -> /Video Controller/VA0
- U49 pad 11: /Video Controller/VA4 -> /Video Controller/VA2
- U49 pad 12: /Video Controller/VA3 -> /Video Controller/VA4
- U49 pad 5: /Video Controller/VA0 -> /Video Controller/VA5
- U49 pad 6: /Video Controller/VA2 -> /Video Controller/VA3
- U50 pad 10: /Video Controller/VA5 -> /Video Controller/VA0
- U50 pad 11: /Video Controller/VA4 -> /Video Controller/VA2
- U50 pad 12: /Video Controller/VA3 -> /Video Controller/VA4
- U50 pad 5: /Video Controller/VA0 -> /Video Controller/VA5
- U50 pad 6: /Video Controller/VA2 -> /Video Controller/VA3
- U51 pad 10: /Video Controller/VA5 -> /Video Controller/VA0
- U51 pad 11: /Video Controller/VA4 -> /Video Controller/VA2
- U51 pad 12: /Video Controller/VA3 -> /Video Controller/VA4
- U51 pad 5: /Video Controller/VA0 -> /Video Controller/VA5
- U51 pad 6: /Video Controller/VA2 -> /Video Controller/VA3
- U52 pad 10: /Video Controller/VA5 -> /Video Controller/VA0
- U52 pad 11: /Video Controller/VA4 -> /Video Controller/VA2
- U52 pad 12: /Video Controller/VA3 -> /Video Controller/VA4
- U52 pad 5: /Video Controller/VA0 -> /Video Controller/VA5
- U52 pad 6: /Video Controller/VA2 -> /Video Controller/VA3
- U53 pad 10: /Video Controller/VA5 -> /Video Controller/VA0
- U53 pad 11: /Video Controller/VA4 -> /Video Controller/VA2
- U53 pad 12: /Video Controller/VA3 -> /Video Controller/VA4
- U53 pad 5: /Video Controller/VA0 -> /Video Controller/VA5
- U53 pad 6: /Video Controller/VA2 -> /Video Controller/VA3
Routing:
- net VCC5V: track 0.00 -> 3273.5 mm, vias 0 -> 6
- net VSS: track 0.00 -> 2619.2 mm, vias 0 -> 16
- net /PD7: track 0.00 -> 568.9 mm, vias 0 -> 9
- net /PD3: track 0.00 -> 559.6 mm, vias 0 -> 8
- net /PD0: track 0.00 -> 557.1 mm, vias 0 -> 9
- net /PD2: track 0.00 -> 556.6 mm, vias 0 -> 8
- net /PD1: track 0.00 -> 554.9 mm, vias 0 -> 8
- net /PD6: track 0.00 -> 553.0 mm, vias 0 -> 8
- net /PD5: track 0.00 -> 550.8 mm, vias 0 -> 9
- net /PD4: track 0.00 -> 538.9 mm, vias 0 -> 8
- net /CPU/R~{W}B: track 0.00 -> 498.0 mm, vias 0 -> 10
- net /CPU/~{IRQ}: track 0.00 -> 468.0 mm, vias 0 -> 9
- net /Video Controller/~{VCAS}: track 0.00 -> 435.8 mm, vias 0 -> 5
- net /PA0: track 0.00 -> 407.8 mm, vias 0 -> 9
- net /CPU/EB: track 0.00 -> 403.1 mm, vias 0 -> 9
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Other:
- board outline added: 450 x 160 mm

Commit message: power traces wip..
Parts:
- moved R15 13.0 mm to (89.9, 243.3), turned to 90 degrees
- moved R8 12.9 mm to (89.9, 211.6), turned to 90 degrees
- moved R3 12.8 mm to (89.9, 182.4), turned to 90 degrees
- moved J6 10.7 mm to (302.0, 142.1)
- moved C59 5.24 mm to (148.1, 277.6), turned to 0 degrees
- moved C57 4.91 mm to (163.6, 277.6), turned to 0 degrees
- moved C55 4.80 mm to (178.9, 277.6), turned to 0 degrees
- moved R18 0.68 mm to (97.6, 261.4)
- moved R19 0.62 mm to (84.6, 261.4)
- moved C58 0.55 mm to (156.0, 277.6)
- moved J10 0.52 mm to (119.8, 141.9)
- moved C10 0.51 mm to (354.8, 172.3)
- moved C62 0.51 mm to (125.5, 277.6)
- moved R17 0.44 mm to (93.7, 256.3)
- moved Q5 0.43 mm to (84.9, 228.1)
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Routing:
- net VEE5V: track 136.2 -> 612.7 mm, vias 1 -> 6
- net /Video Controller/ANA_SYNC: track 0.00 -> 170.4 mm
- net /Sound/LIGHTPEN_SWITCH: track 0.00 -> 143.3 mm, vias 0 -> 1
- net /Video Controller/TTL_LUM: track 0.00 -> 135.1 mm, vias 0 -> 1
- net /Video Controller/TTL_B: track 0.00 -> 132.1 mm, vias 0 -> 1
- net /Video Controller/ANA_B: track 0.00 -> 131.2 mm
- net /Video Controller/TTL_SYNC: track 0.00 -> 129.5 mm, vias 0 -> 1
- net /Sound/JOY2_RIGHT: track 0.00 -> 117.2 mm, vias 0 -> 1
- net /Sound/JOY2_LEFT: track 0.00 -> 112.1 mm, vias 0 -> 1
- net /Video Controller/ANA_G: track 0.00 -> 98.4 mm
- net VCC5V: track 3273.5 -> 3357.4 mm, vias 6 -> 7
- net Net-(U37-Qh): track 0.00 -> 79.4 mm, vias 0 -> 2
- net /Video Controller/TTL_R: track 30.7 -> 109.5 mm
- net VCC12V: track 60.5 -> 137.5 mm, vias 0 -> 1
- net /Video Controller/ANA_R: track 0.00 -> 71.4 mm
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- added copper zone on B.Cu, net VCC12V
- added copper zone on F.Cu, net VCC12V
- added copper zone on B.Cu, net VCC5V
- added copper zone on F.Cu, net VEE5V
- added copper zone on F.Cu, net VSS

Commit message: some footprints fixes and minor changes.
Parts:
- J3: footprint Connector_Dsub:DSUB-15_Socket_Horizontal_P2.77x2.84mm_EdgePinOffset9.40mm -> Connector_Dsub:DSUB-15_Pins_Horizontal_P2.77x2.84mm_EdgePinOffset9.40mm; moved to F.Cu
- J6: footprint Connector_Dsub:DSUB-9_Pins_Horizontal_P2.77x2.54mm_EdgePinOffset9.40mm -> Connector_Dsub:DSUB-9_Socket_Horizontal_P2.77x2.54mm_EdgePinOffset9.40mm
- moved J6 10.6 mm to (291.4, 142.2)
- moved J3 0.23 mm to (441.5, 142.3), turned to 180 degrees
Connections:
- U2 pad 24: unconnected-(U2-VCC-Pad24) -> VCC5V
Routing:
- net /ROM_pack/RP_D2: track 0.00 -> 67.0 mm, vias 0 -> 1
- net /ROM_pack/RP_D4: track 0.00 -> 64.8 mm
- net /ROM_pack/RP_D1: track 0.00 -> 64.0 mm, vias 0 -> 1
- net /ROM_pack/RP_D3: track 0.00 -> 63.0 mm, vias 0 -> 1
- net /ROM_pack/RP_D0: track 0.00 -> 63.0 mm
- net /ROM_pack/RP_D5: track 0.00 -> 62.1 mm
- net /ROM_pack/RP_D7: track 0.00 -> 58.0 mm
- net VSS: track 2614.4 -> 2670.7 mm
- net /ROM_pack/RP_A11: track 0.00 -> 38.9 mm
- net /ROM_pack/RP_A10: track 0.00 -> 30.1 mm
- net /ROM_pack/RP_A8: track 0.00 -> 28.9 mm
- net /ROM_pack/RP_A9: track 0.00 -> 27.0 mm
- net /ROM_pack/RP_A2: track 0.00 -> 23.8 mm
- net /ROM_pack/RP_A0: track 0.00 -> 22.5 mm
- net /ROM_pack/RP_A3: track 16.1 -> 37.6 mm
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
Commit message: Fix footprints and many drc errors.
Parts:
- added J1: Conn_01x06_Socket, TerminalBlock_CUI:TerminalBlock_CUI_TB007-508-06_1x06_P5.08mm_Horizontal, F.Cu at (519.7, 201.7)
- D1, D2, D3: footprint Diode_THT:D_DO-35_SOD27_P7.62mm_Horizontal -> Diode_THT:D_DO-35_SOD27_P12.70mm_Horizontal
- J2: footprint Connector_PinSocket_2.54mm:PinSocket_2x20_P2.54mm_Vertical -> Library:Ribbon_Conn
- J5, J9: footprint Connector_PinHeader_2.54mm:PinHeader_1x05_P2.54mm_Vertical -> Library:DIN5-RA-PTH
- moved J9 13.1 mm to (186.7, 131.8), turned to 180 degrees
- moved J5 12.6 mm to (330.7, 131.8), turned to 180 degrees
- moved J2 0.25 mm to (518.2, 142.0)
- moved D3 0.19 mm to (504.2, 224.5)
Routing:
- net VCC12V: track 137.5 -> 661.9 mm
- net VEE5V: track 612.7 -> 887.9 mm
- net VCC5V: track 3359.0 -> 3488.4 mm
- net VSS: track 2670.7 -> 2757.0 mm
- net /Tape-Modem/OUT_50mV_LEVEL: track 15.2 -> 24.1 mm
- net /ROM_pack/RP_D4: track 64.8 -> 72.2 mm
- net /CPU/Q: track 148.9 -> 156.3 mm
- net /ROM_pack/RP_A11: track 38.9 -> 46.1 mm
- net /Video Controller/~{D_{3}I}: track 169.9 -> 177.1 mm
- net /ROM_pack/RP_A0: track 22.5 -> 29.4 mm
- net /ROM_pack/RP_D0: track 63.0 -> 69.9 mm
- net /ROM_pack/RP_D6: track 60.3 -> 67.0 mm
- net /ROM_pack/RP_D2: track 67.0 -> 73.4 mm
- net /ROM_pack/RP_A8: track 28.9 -> 35.0 mm
- net /ROM_pack/RP_A2: track 23.8 -> 29.7 mm
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Other:
- board text added: "001 A"
- board text added: "APOLLO 7"
- board text added: "SQUALE"
