File: hardware/Motherboard/Squale.kicad_pcb (KiCad board)
At the start: 2 copper layers, 450 x 160 mm, 219 parts, among them J1 Conn_01x06_Socket, J10 DA15_Socket, J11 Conn_01x22_Socket, J2 Conn_02x20_Odd_Even, J3 DA15_Socket, J4 DB25_Socket, J5 DIN-5_180degree, J6 DE9_Socket, J7 DE9_Pins, J8 DE9_Pins, J9 DIN-5_180degree, P1 VR10K, Q1 2N2222, Q2 2N2222, Q3 2N2222, Q4 2N2222, Q5 2N2222, Q6 2N2222, Q7 2N2222, U1 MC6809, U10 74LS138, U11 74LS245, U12 74LS541, U13 74LS541, U14 74LS541, U15 74LS393, U16 MK4164N, U17 MK4164N, U18 MK4164N, U19 MK4164N, U2 27C32, U20 MK4164N, U21 MK4164N, U22 MK4164N, U23 MK4164N, U24 74LS123, U25 74LS74, U26 74LS74, U28 74LS04, U29 74LS02, U3 74LS245, U30 74LS245, U31 74LS541, U32 74LS04, U33 74LS17, U34 74LS166, U35 74LS166, U36 74LS166, U37 74LS166, U38 MK4116N, U39 MK4116N, U4 74LS139, U40 MK4116N, U41 MK4116N, U42 MK4116N, U43 MK4116N, U44 MK4116N, U45 MK4116N, U46 MK4116N, U47 MK4116N, U48 MK4116N, U49 MK4116N, U5 74LS20, U50 MK4116N, U51 MK4116N, U52 MK4116N, U53 MK4116N, U54 74LS374, U55 74LS374, U56 74LS541, U57 74LS32, U58 74LS374, U59 EF9365, U6 74LS08, U60 74LS04, U61 74LS193, U62 TBP18S030N, U63 74LS32, U64 74LS374, U65 AY-3-8910A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

Commit message: more fixes !
Parts:
- U2: footprint Package_DIP:DIP-24_18.0mmx34.29mm_W15.24mm -> Package_DIP:DIP-24_W15.24mm_Socket
Routing:
- net VCC5V: track 3488.4 -> 3476.3 mm
Changed lines of the file:
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@@
 		(sheetname "/DRAM/")
 		(sheetfile "DRAM.kicad_sch")
-		(attr through_hole)
+		(attr through_hole dnp)
 		(fp_line
 			(start 7.12 1.37)
@@
 		)
 	)
-	(footprint "Package_DIP:DIP-24_18.0mmx34.29mm_W15.24mm"
+	(footprint "Package_DIP:DIP-24_W15.24mm_Socket"
 		(layer "F.Cu")
 		(at 450.85 232.156 180)
-		(descr "24-lead though-hole mounted DIP package, row spacing 15.24 mm (600 mils) https://www.mouser.at/datasheet/2/389/m48t02-1849963.pdf")
-		(tags "THT DIP DIL PDIP 2.54mm 15.24mm 600mil PCDIP24 CAPHAT M48T02 M48T12 M48Z02 M48Z12")
+		(descr "24-lead though-hole mounted DIP package, row spacing 15.24mm (600 mils), Socket")
+		(tags "THT DIP DIL PDIP 2.54mm 15.24mm 600mil Socket")
 		(property "Reference" "U2"
-			(at 7.62 -4.46 180)
+			(at 7.62 -2.33 180)
 			(layer "F.SilkS")
 			(effects
@@
 		(property "Datasheet" ""
 			(at 0 0 180)
-			(unlocked yes)
 			(layer "F.Fab")
 			(hide yes)
@@
 		(property "Description" ""
 			(at 0 0 180)
-			(unlocked yes)
 			(layer "F.Fab")
 			(hide yes)
@@
 		(attr through_hole)
 		(fp_line
-			(start 16.62 31.115)
-			(end 16.62 -3.175)
+			(start 14.08 29.27)
+			(end 14.08 -1.33)
 			(stroke
 				(width 0.12)
@@
 		)
 		(fp_line
-			(start 16.62 -3.175)
-			(end 8.62 -3.175)
+			(start 14.08 -1.33)
+			(end 8.62 -1.33)
 			(stroke
 				(width 0.12)
@@
 		)
 		(fp_line
-			(start 6.62 -3.175)
-			(end -1.38 -3.175)
+			(start 6.62 -1.33)
+			(end 1.16 -1.33)
 			(stroke
 				(width 0.12)
@@
 		)
 		(fp_line
-			(start -1.38 31.115)
-			(end 16.62 31.115)
+			(start 1.16 29.27)
+			(end 14.08 29.27)
 			(stroke
 				(width 0.12)
@@
 		)
 		(fp_line
-			(start -1.38 -3.175)
-			(end -1.38 31.115)
+			(start 1.16 -1.33)
+			(end 1.16 29.27)
+			(stroke
+				(width 0.12)
+				(type solid)
+			)
+			(layer "F.SilkS")
+		)
+		(fp_rect
+			(start -1.33 -1.39)
+			(end 16.57 29.33)
 			(stroke
 				(width 0.12)
 				(type solid)
 			)
+			(fill no)
 			(layer "F.SilkS")
 		)
 		(fp_arc
-			(start 8.62 -3.175)
-			(mid 7.62 -2.175)
-			(end 6.62 -3.175)
+			(start 8.62 -1.33)
+			(mid 7.62 -0.33)
+			(end 6.62 -1.33)
 			(stroke
 				(width 0.12)
@@
 		)
 		(fp_rect
-			(start -1.63 -3.43)
-			(end 16.87 31.37)
+			(start -1.53 -1.58)
+			(end 16.77 29.53)
 			(stroke
 				(width 0.05)
-				(type default)
+				(type solid)
 			)
 			(fill no)
@@
 			(layer "F.Fab")
 		)
+		(fp_rect
+			(start -1.27 -1.33)
+			(end 16.51 29.27)
+			(stroke
+				(width 0.1)
+				(type solid)
+			)
+			(fill no)
+			(layer "F.Fab")
+		)
 		(fp_text user "${REFERENCE}"
-			(at 7.62 13.97 180)
+			(at 7.62 13.97 270)
 			(layer "F.Fab")
 			(effects
@@
 			)
 		)
-		(pad "1" thru_hole rect
+		(pad "1" thru_hole roundrect
 			(at 0 0 180)
 			(size 1.6 1.6)
@@
 			(layers "*.Cu" "*.Mask")
 			(remove_unused_layers no)
+			(roundrect_rratio 0.15625)
 			(net 184 "/A7")
 			(pinfunction "A7")
 			(pintype "input")
 		)
-		(pad "2" thru_hole oval
+		(pad "2" thru_hole circle
 			(at 0 2.54 180)
 			(size 1.6 1.6)
@@
 			(pintype "input")
 		)
-		(pad "3" thru_hole oval
+		(pad "3" thru_hole circle
 			(at 0 5.08 180)
 			(size 1.6 1.6)
@@
 			(pintype "input")
 		)
-		(pad "4" thru_hole oval
+		(pad "4" thru_hole circle
 			(at 0 7.62 180)
 			(size 1.6 1.6)
@@
 			(pintype "input")
 		)
-		(pad "5" thru_hole oval
+		(pad "5" thru_hole circle
 			(at 0 10.16 180)
 			(size 1.6 1.6)
@@
 			(pintype "input")
 		)
-		(pad "6" thru_hole oval
+		(pad "6" thru_hole circle
 			(at 0 12.7 180)
 			(size 1.6 1.6)
@@
 			(pintype "input")
 		)
-		(pad "7" thru_hole oval
+		(pad "7" thru_hole circle
 			(at 0 15.24 180)
 			(size 1.6 1.6)
@@
 			(pintype "input")
 		)
-		(pad "8" thru_hole oval
+		(pad "8" thru_hole circle
 			(at 0 17.78 180)
 			(size 1.6 1.6)
@@
 			(pintype "input")
 		)
-		(pad "9" thru_hole oval
+		(pad "9" thru_hole circle
 			(at 0 20.32 180)
 			(size 1.6 1.6)
@@
 			(pintype "bidirectional")
 		)
-		(pad "10" thru_hole oval
+		(pad "10" thru_hole circle
 			(at 0 22.86 180)
 			(size 1.6 1.6)
@@
 			(pintype "bidirectional")
 		)
-		(pad "11" thru_hole oval
+		(pad "11" thru_hole circle
 			(at 0 25.4 180)
 			(size 1.6 1.6)
@@
 			(pintype "bidirectional")
 		)
-		(pad "12" thru_hole oval
+		(pad "12" thru_hole circle
 			(at 0 27.94 180)
 			(size 1.6 1.6)
@@
 			(pintype "power_in")
 		)
-		(pad "13" thru_hole oval
+		(pad "13" thru_hole circle
 			(at 15.24 27.94 180)
 			(size 1.6 1.6)
@@
 			(pintype "bidirectional")
 		)
-		(pad "14" thru_hole oval
+		(pad "14" thru_hole circle
 			(at 15.24 25.4 180)
 			(size 1.6 1.6)
@@
 			(pintype "bidirectional")
 		)
-		(pad "15" thru_hole oval
+		(pad "15" thru_hole circle
 			(at 15.24 22.86 180)
 			(size 1.6 1.6)
@@
 			(pintype "bidirectional")
 		)
-		(pad "16" thru_hole oval
+		(pad "16" thru_hole circle
 			(at 15.24 20.32 180)
 			(size 1.6 1.6)
@@
 			(pintype "bidirectional")
 		)
-		(pad "17" thru_hole oval
+		(pad "17" thru_hole circle
 			(at 15.24 17.78 180)
 			(size 1.6 1.6)
@@
 			(pintype "bidirectional")
 		)
-		(pad "18" thru_hole oval
+		(pad "18" thru_hole circle
 			(at 15.24 15.24 180)
 			(size 1.6 1.6)
@@
 			(pintype "input")
 		)
-		(pad "19" thru_hole oval
+		(pad "19" thru_hole circle
 			(at 15.24 12.7 180)
 			(size 1.6 1.6)
@@
 			(pintype "input")
 		)
-		(pad "20" thru_hole oval
+		(pad "20" thru_hole circle
 			(at 15.24 10.16 180)
 			(size 1.6 1.6)
@@
 			(pintype "input")
 		)
-		(pad "21" thru_hole oval
+		(pad "21" thru_hole circle
 			(at 15.24 7.62 180)
 			(size 1.6 1.6)
@@
 			(pintype "input")
 		)
-		(pad "22" thru_hole oval
+		(pad "22" thru_hole circle
 			(at 15.24 5.08 180)
 			(size 1.6 1.6)
@@
 			(pintype "input")
 		)
-		(pad "23" thru_hole oval
+		(pad "23" thru_hole circle
 			(at 15.24 2.54 180)
 			(size 1.6 1.6)
@@
 			(pintype "input")
 		)
-		(pad "24" thru_hole oval
+		(pad "24" thru_hole circle
 			(at 15.24 0 180)
 			(size 1.6 1.6)
@@
 			(pintype "power_in")
 		)
-		(group ""
-			(members "04b4fc87-26b6-45a5-81f2-581aca534fd8" "24ce0c3a-da4a-4da2-a691-6d933f09457b"
-				"47270219-97cb-463a-967f-0ee7693b1b35" "4c07ae77-cebb-4cc5-a106-1562e4dd7e0e"
-				"9ae99df5-d1b8-4df3-ab3e-50f2b5e4c08f" "a1e215c7-3d0d-484d-afe8-9e7bd7603fa1"
-				"dff478cd-6f91-4fbd-a5e3-d09cdaa2f98c"
-			)
-		)
 		(embedded_fonts no)
-		(model "${KICAD9_3DMODEL_DIR}/Package_DIP.3dshapes/DIP-24_18.0mmx34.29mm_W15.24mm.step"
+		(model "${KICAD9_3DMODEL_DIR}/Package_DIP.3dshapes/DIP-24_W15.24mm_Socket.step"
 			(offset
 				(xyz 0 0 0)
@@
 	)
 	(segment
-		(start 496.824 194.818)
-		(end 492.76 198.882)
-		(width 0.3175)
-		(layer "B.Cu")
-		(net 1)
-	)
-	(segment
 		(start 91.186 191.516)
 		(end 91.165641 191.536359)
@@
 		(width 0.3175)
 		(layer "B.Cu")
-		(net 1)
-	)
-	(segment
-		(start 492.76 198.882)
-		(end 492.76 205.232)
-		(width 0.3175)
-		(layer "B.Cu")

Commit message: connection fix + power line width.
Connections:
- U69 pad 11: /PA[6..0] -> /PA0
Routing:
- net VSS: track 2757.0 -> 2764.3 mm
- net /A8: track 85.9 -> 82.9 mm
- net /PA0: track 407.8 -> 410.7 mm
- net /Video Controller/VA5: track 331.4 -> 330.6 mm
- net VEE5V: track 887.9 -> 887.1 mm
- net /Video Controller/TTL_LUM: track 135.1 -> 134.4 mm
- net Net-(U25A-~{S}): track 177.7 -> 177.1 mm
- net Net-(U67D--): track 27.2 -> 26.6 mm
- net /PA5: track 110.0 -> 109.5 mm
- net /PD2: track 556.6 -> 556.1 mm
- net /DRAM/VMA: track 264.0 -> 263.5 mm
- net /Tape-Modem/IN_1: vias 1 -> 0
- net /CPU/~{RST}: vias 5 -> 4
Other:
- board text added: "APOLLO 7 -"

Commit message: more minor fixes.
Parts:
- moved U61 0.36 mm to (258.3, 223.0)
- moved U4 0.12 mm to (403.9, 233.4)
Routing:
- net VCC5V: track 3476.4 -> 3474.2 mm
- net VSS: track 2764.3 -> 2762.1 mm
- net /Sound/SOUND_OUT: track 30.8 -> 30.0 mm
- net /Keyboard/KEYB_R2: track 24.9 -> 24.1 mm
- net /Video Controller/W1: track 148.6 -> 147.8 mm
- net /CPU/~{RST}: track 325.0 -> 324.3 mm
- net /DRAM/RA7: track 175.2 -> 174.5 mm
- net Net-(U34-Qh): track 39.8 -> 39.2 mm
- net /Video Controller/TTL_R: track 109.5 -> 108.9 mm
- net Net-(U25A-C): track 179.0 -> 178.5 mm
- net Net-(U24A-~{Q}): track 30.8 -> 30.3 mm
- net /Video Controller/~{D_{1}V}: track 134.6 -> 134.0 mm
- net Net-(U70-Pad1): track 14.7 -> 14.2 mm
- net /Video Controller/~{D_{0}I}: track 154.2 -> 153.7 mm

Commit message: fixes
Parts:
- moved C71 0.27 mm to (125.5, 159.6)
Connections:
- U34 pad 7: unconnected-(U34-Clk-Pad7) -> VSS
- U35 pad 7: unconnected-(U35-Clk-Pad7) -> VSS
- U36 pad 7: unconnected-(U36-Clk-Pad7) -> VSS
- U37 pad 7: unconnected-(U37-Clk-Pad7) -> VSS
Routing:
- net VSS: track 2762.1 -> 2770.3 mm
- net VCC5V: track 3474.2 -> 3472.9 mm
- net /Video Controller/VA4: track 333.0 -> 333.7 mm
