File: hardware/SS30_Floppy_Disk_Controller/SS30_Floppy_Disk_Controller.kicad_sch (KiCad schematic)
At the start: 18 parts, among them IC1 WD1770, U1 74LS06, U2 74LS06, U3 6821, U4 74LS02

Commit message: WIP : schematic
Parts:
- removed unit 2 of U1
- removed unit 2 of U2
- removed unit 6 of U2
- added C? (x5): 100nF, symbol Device:C
- added R? (x3): 220, symbol Device:R
- added unit 6 of U4
- added unit 2 of U4
- added unit 2 of U5
- added U?: LM7805_TO220, Package_TO_SOT_THT:TO-220-3_Vertical, symbol Regulator_Linear:LM7805_TO220
- R?: value R -> 220
- gave numbers to parts that had none: 2
- renumbered IC1 to U1, U3 to U2, U4 to U3, U2 to U4, U1 to U5
Connections:
- net A0: now also U1.3 (A0), U2.36 (RS0)
- net A1: now also U1.4 (A1), U2.35 (RS1)
- net VCC5V: now also U2.20 (VCC), C?.1, C?.1, C?.1, C?.1, R?.1, R?.1, R?.1, U?.3 (VO)
- net VCC8V: now also C?.1, U?.1 (VI)
- net VSS: now also C?.2, C?.2, C?.2, C?.2, C?.2, U?.2 (GND)
- net ~{DS1}: now also U4.4
- net ~{DS2}: now also J?.14 (Pin_14), U4.12; no longer J?.6 (Pin_6), U4.2
- net ~{MON}: now also J?.16 (Pin_16), U5.4; no longer J?.14 (Pin_14)
- net ~{CS_WD}: now reaches U1.1 (~{CS}), U3.1
- net at U1.16 (STEP): now also U5.9
- net at U1.17 (DIRC): now also U5.5
- net CLK_8MHZ: now reaches R?.2, U1.18 (CLK), U3.13, Y?.2
- net ~{RDATA_RETIMED}: now reaches U1.19 (~{RD}), U6.1 (~{Q})
- net at U1.20 (MO): now also U5.3
- net at U1.21 (WG): now also U5.13
- net at U1.22 (WD): now also U5.1
- net ~{TRK00}: now reaches U1.23 (~{TR00})
- net ~{TRK00}: now also J?.26 (Pin_26), R?.2
- net ~{INDEX}: now reaches U1.24 (~{IP})
- net ~{INDEX}: now also J?.8 (Pin_8), R?.2
- net ~{WPROTECT}: now reaches U1.25 (~{WPRT})
- net ~{WPROTECT}: now also J?.28 (Pin_28), R?.2
- net ~{DDEN}: now reaches U1.26 (~{DDEN}), U2.15 (PB5)
- net ~{STEP}: now reaches U5.8
- net ~{STEP}: now also J?.20 (Pin_20)
- net DS1: now reaches U2.12 (PB2)
- net DS1: now also U4.3
- net DS3: now reaches U2.10 (PB0), U4.1
- net DS2: now reaches U2.11 (PB1)
- net DS2: now also U4.13
- net DS0: now reaches U2.13 (PB3), U4.5
- net SIDE1: now reaches U2.14 (PB4), U4.9
- net ~{DIR}: now reaches J?.18 (Pin_18)
- net ~{DIR}: now also U5.6
- net ~{WDATA}: now reaches J?.22 (Pin_22)
- net ~{WDATA}: now also U5.2
- net ~{WGATE}: now reaches J?.24 (Pin_24)
- net ~{WGATE}: now also U5.12
- new net ~{DS3}: J?.6 (Pin_6), U4.2
- no-connect marks 33 -> 37
Other:
- note added: "Base : 0x0"
- note added: "Base : 0x8"
- moved on the sheet: C?, J?, R?, U1, U2, U3A, U3B, U3C, U3D, U3E, U4A, U4C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

Commit message: WIP : annotation.
Parts:
- gave numbers to parts that had none: 3
Changed lines of the file:
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@@
 		(dnp no)
 		(fields_autoplaced yes)
-		(property "Reference" "U?"
+		(property "Reference" "U7"
 			(at 99.06 20.32 0)
 			(effects
@@
 			(project ""
 				(path "/84fa1d29-30c9-43d1-87fc-482896eea75d"
-					(reference "U?")
+					(reference "U7")
 					(unit 1)
 				)
@@
 		(on_board yes)
 		(dnp no)
-		(property "Reference" "J?"
+		(property "Reference" "J2"
 			(at 300.99 125.73 0)
 			(effects
@@
 			(project ""
 				(path "/84fa1d29-30c9-43d1-87fc-482896eea75d"
-					(reference "J?")
+					(reference "J2")
 					(unit 1)
 				)
@@
 		(on_board yes)
 		(dnp no)
-		(property "Reference" "J?"
+		(property "Reference" "J1"
 			(at 50.8 93.9799 0)
 			(effects
@@
 			(project ""
 				(path "/84fa1d29-30c9-43d1-87fc-482896eea75d"
-					(reference "J?")
-					(unit 1)
-				)
+					(reference "J1")
+					(unit 1)
+				)

Commit message: WIP : annotation.
Parts:
- gave numbers to parts that had none: 17
Other:
- note added: "SS-30 Bus"
- moved on the sheet: U3A, U3B
Changed lines of the file:
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@@
 		)
 	)
+	(text "SS-30 Bus"
+		(exclude_from_sim no)
+		(at 54.102 53.848 0)
+		(effects
+			(font
+				(size 1.27 1.27)
+			)
+		)
+	)
 	(text "Base : 0x0"
 		(exclude_from_sim no)
@@
 	)
 	(junction
-		(at 139.7 132.08)
+		(at 143.51 132.08)
 		(diameter 0)
 		(color 0 0 0 0)
@@
 	(wire
 		(pts
-			(xy 121.92 134.62) (xy 106.68 134.62)
-		)
-		(stroke
-			(width 0)
-			(type default)
-		)
-	)
-	(wire
-		(pts
 			(xy 156.21 199.39) (xy 177.8 199.39)
 		)
@@
 	(wire
 		(pts
-			(xy 137.16 132.08) (xy 139.7 132.08)
+			(xy 140.97 132.08) (xy 143.51 132.08)
 		)
 		(stroke
@@
 	(wire
 		(pts
-			(xy 109.22 129.54) (xy 121.92 129.54)
+			(xy 109.22 129.54) (xy 125.73 129.54)
 		)
 		(stroke
@@
 	(wire
 		(pts
-			(xy 139.7 132.08) (xy 139.7 134.62)
+			(xy 143.51 132.08) (xy 143.51 134.62)
 		)
 		(stroke
@@
 	(wire
 		(pts
-			(xy 139.7 129.54) (xy 139.7 132.08)
+			(xy 143.51 129.54) (xy 143.51 132.08)
+		)
+		(stroke
+			(width 0)
+			(type default)
+		)
+	)
+	(wire
+		(pts
+			(xy 106.68 134.62) (xy 125.73 134.62)
 		)
 		(stroke
@@
 	(wire
 		(pts
-			(xy 154.94 132.08) (xy 158.75 132.08)
-		)
-		(stroke
-			(width 0)
-			(type default)
-		)
-	)
-	(wire
-		(pts
 			(xy 203.2 199.39) (xy 213.36 199.39)
 		)
@@
 		)
 	)
+	(label "~{IO_SELECT}"
+		(at 116.84 134.62 0)
+		(effects
+			(font
+				(size 1.27 1.27)
+			)
+			(justify left bottom)
+		)
+	)
 	(label "~{DS1}"
 		(at 288.29 144.78 0)
@@
 		(dnp no)
 		(fields_autoplaced yes)
-		(property "Reference" "C?"
+		(property "Reference" "C5"
 			(at 118.11 29.2099 0)
 			(effects
@@
 			(project ""
 				(path "/84fa1d29-30c9-43d1-87fc-482896eea75d"
-					(reference "C?")
+					(reference "C5")
 					(unit 1)
 				)
@@
 		(dnp no)
 		(fields_autoplaced yes)
-		(property "Reference" "R?"
+		(property "Reference" "R7"
 			(at 266.7 157.4799 0)
 			(effects
@@
 			(project ""
 				(path "/84fa1d29-30c9-43d1-87fc-482896eea75d"
-					(reference "R?")
+					(reference "R7")
 					(unit 1)
 				)
@@
 		(dnp no)
 		(fields_autoplaced yes)
-		(property "Reference" "Y?"
+		(property "Reference" "Y1"
 			(at 66.04 187.96 0)
 			(effects
@@
 			(project ""
 				(path "/84fa1d29-30c9-43d1-87fc-482896eea75d"
-					(reference "Y?")
+					(reference "Y1")
 					(unit 1)
 				)
@@
 		(dnp no)
 		(fields_autoplaced yes)
-		(property "Reference" "R?"
+		(property "Reference" "R4"
 			(at 232.41 219.7099 0)
 			(effects
@@
 			(project ""
 				(path "/84fa1d29-30c9-43d1-87fc-482896eea75d"
-					(reference "R?")
+					(reference "R4")
 					(unit 1)
 				)
@@
 		(on_board yes)
 		(dnp no)
-		(property "Reference" "C?"
+		(property "Reference" "C2"
 			(at 40.894 200.66 90)
 			(effects
@@
 			(project "SS30_Floppy_Disk_Controller"
 				(path "/84fa1d29-30c9-43d1-87fc-482896eea75d"
-					(reference "C?")
+					(reference "C2")
 					(unit 1)
 				)
@@
 		(dnp no)
 		(fields_autoplaced yes)
-		(property "Reference" "C?"
+		(property "Reference" "C7"
 			(at 246.38 30.4799 0)
 			(effects
@@
 			(project "SS30_Floppy_Disk_Controller"
 				(path "/84fa1d29-30c9-43d1-87fc-482896eea75d"
-					(reference "C?")
+					(reference "C7")
 					(unit 1)
 				)
@@
 		(dnp no)
 		(fields_autoplaced yes)
-		(property "Reference" "R?"
+		(property "Reference" "R2"
 			(at 53.34 200.66 90)
 			(effects
@@
 			(project "SS30_Floppy_Disk_Controller"
 				(path "/84fa1d29-30c9-43d1-87fc-482896eea75d"
-					(reference "R?")
+					(reference "R2")
 					(unit 1)
 				)
@@
 		(dnp no)
 		(fields_autoplaced yes)
-		(property "Reference" "C?"
+		(property "Reference" "C6"
 			(at 210.82 30.4799 0)
 			(effects
@@
 			(project "SS30_Floppy_Disk_Controller"
 				(path "/84fa1d29-30c9-43d1-87fc-482896eea75d"
-					(reference "C?")
+					(reference "C6")
 					(unit 1)
 				)
@@
 	(symbol
 		(lib_id "74xx:74LS02")
-		(at 129.54 132.08 0)
+		(at 133.35 132.08 0)
 		(unit 2)
 		(exclude_from_sim no)
@@
 		(fields_autoplaced yes)
 		(property "Reference" "U3"
-			(at 129.54 123.19 0)
+			(at 133.35 123.19 0)
 			(effects
 				(font
@@
 		)
 		(property "Value" "74LS02"
-			(at 129.54 125.73 0)
+			(at 133.35 125.73 0)
 			(effects
 				(font
@@
 		)
 		(property "Footprint" ""
-			(at 129.54 132.08 0)
+			(at 133.35 132.08 0)
 			(effects
 				(font
@@
 		)
 		(property "Datasheet" "http://www.ti.com/lit/gpn/sn74ls02"
-			(at 129.54 132.08 0)
+			(at 133.35 132.08 0)
 			(effects
 				(font
@@
 		)
 		(property "Description" "quad 2-input NOR gate"
-			(at 129.54 132.08 0)
+			(at 133.35 132.08 0)
 			(effects
 				(font
@@
 		(dnp no)
 		(fields_autoplaced yes)
-		(property "Reference" "R?"
+		(property "Reference" "R5"
 			(at 266.7 134.6199 0)
 			(effects
@@
 			(project "SS30_Floppy_Disk_Controller"
 				(path "/84fa1d29-30c9-43d1-87fc-482896eea75d"
-					(reference "R?")
+					(reference "R5")
 					(unit 1)
 				)
@@
 	(symbol
 		(lib_id "74xx:74LS02")
-		(at 147.32 132.08 0)
+		(at 151.13 132.08 0)
 		(unit 1)
 		(exclude_from_sim no)
@@
 		(fields_autoplaced yes)
 		(property "Reference" "U3"
-			(at 147.32 123.19 0)
+			(at 151.13 123.19 0)
 			(effects
 				(font
@@
 		)
 		(property "Value" "74LS02"
-			(at 147.32 125.73 0)
+			(at 151.13 125.73 0)
 			(effects
 				(font
@@
 		)
 		(property "Footprint" ""
-			(at 147.32 132.08 0)
+			(at 151.13 132.08 0)
 			(effects
 				(font
@@
 		)
 		(property "Datasheet" "http://www.ti.com/lit/gpn/sn74ls02"
-			(at 147.32 132.08 0)
+			(at 151.13 132.08 0)
 			(effects
 				(font
@@
 		)
 		(property "Description" "quad 2-input NOR gate"
-			(at 147.32 132.08 0)
+			(at 151.13 132.08 0)
 			(effects
 				(font
@@
 		(on_board yes)
 		(dnp no)
-		(property "Reference" "C?"
+		(property "Reference" "C4"
 			(at 87.884 29.464 0)
 			(effects
@@
 			(project "SS30_Floppy_Disk_Controller"
 				(path "/84fa1d29-30c9-43d1-87fc-482896eea75d"
-					(reference "C?")
+					(reference "C4")
 					(unit 1)
 				)
@@
 		(on_board yes)
 		(dnp no)
-		(property "Reference" "R?"
+		(property "Reference" "R1"
 			(at 122.936 77.724 90)
 			(effects
@@
 			(project ""
 				(path "/84fa1d29-30c9-43d1-87fc-482896eea75d"
-					(reference "R?")
+					(reference "R1")
 					(unit 1)
 				)
@@
 		(dnp no)
 		(fields_autoplaced yes)
-		(property "Reference" "R?"
+		(property "Reference" "R6"
 			(at 259.08 157.4799 0)
 			(effects
@@
 			(project "SS30_Floppy_Disk_Controller"
 				(path "/84fa1d29-30c9-43d1-87fc-482896eea75d"
-					(reference "R?")
+					(reference "R6")
 					(unit 1)
 				)
@@
 		(dnp no)
 		(fields_autoplaced yes)
-		(property "Reference" "C?"
+		(property "Reference" "C8"
 			(at 279.4 30.4799 0)
 			(effects
@@
 			(project "SS30_Floppy_Disk_Controller"
 				(path "/84fa1d29-30c9-43d1-87fc-482896eea75d"
-					(reference "C?")
+					(reference "C8")
 					(unit 1)
 				)
@@
 		(dnp no)
 		(fields_autoplaced yes)
-		(property "Reference" "R?"
+		(property "Reference" "R3"
 			(at 80.01 200.66 90)
 			(effects
@@
 			(project "SS30_Floppy_Disk_Controller"
 				(path "/84fa1d29-30c9-43d1-87fc-482896eea75d"
-					(reference "R?")
+					(reference "R3")
 					(unit 1)
 				)
@@
 		(dnp no)
 		(property "Reference" "J1"
-			(at 50.8 93.9799 0)
+			(at 54.61 51.054 0)
 			(effects
 				(font
@@
 		)
 		(property "Value" "Conn_01x30_Socket"
-			(at 50.8 96.5199 0)
+			(at 65.786 136.398 0)
 			(effects
 				(font
@@
 		(on_board yes)
 		(dnp no)
-		(property "Reference" "C?"
+		(property "Reference" "C3"
 			(at 66.294 214.376 90)
 			(effects
@@
 			(project ""
 				(path "/84fa1d29-30c9-43d1-87fc-482896eea75d"
-					(reference "C?")
+					(reference "C3")
 					(unit 1)
 				)
@@
 		(dnp no)
 		(fields_autoplaced yes)
-		(property "Reference" "R?"
+		(property "Reference" "R8"
 			(at 266.7 182.8799 0)
 			(effects
@@
 			(project "SS30_Floppy_Disk_Controller"
 				(path "/84fa1d29-30c9-43d1-87fc-482896eea75d"
-					(reference "R?")
+					(reference "R8")
 					(unit 1)
 				)
@@
 		(dnp no)
 		(fields_autoplaced yes)
-		(property "Reference" "C?"
+		(property "Reference" "C1"
 			(at 233.68 231.1399 0)
 			(effects
@@
 			(project ""
 				(path "/84fa1d29-30c9-43d1-87fc-482896eea75d"
-					(reference "C?")
+					(reference "C1")
 					(unit 1)
 				)

Commit message: fix some missing values.
Parts:
- added C9: 22uF, symbol Device:C_Polarized
- C1: value C -> 100 pF
- C2: value C -> 22 pF
- C3: value C -> 10nF
- R4: value R -> 4K7
Connections:
- net VCC5V: now also C9.1
- net VSS: now also C9.2
Other:
- moved on the sheet: C2, C3, C4, C5, R2, R3, U3C, U3D, U7, Y1

Commit message: comment/notes added.
Other:
- note added: "4,7Kohms × 100pF × 0,7 = 329 ns"
- note added: "8MHz clock source"
- note added: "Drive, head and density selection port"
- note added: "Floppy controller"
- note added: "Floppy interface drivers"
- note added: "Incoming read data pulses duration correction/Standardization"
- note added: "SS30 8V to 5V power supply"
- moved on the sheet: C6, C7, C8, U3A, U3B, U3E, U4G, U5G

Commit message: port -> register
Other:
- note added: "Drive, head and density selectors register"
- note removed: "Drive, head and density selection port"
Changed lines of the file:
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@@
 		)
 	)
-	(text "Drive, head \nand density \nselection port"
+	(text "Drive, head \nand density \nselectors register"
 		(exclude_from_sim no)
-		(at 165.354 32.512 0)
+		(at 169.418 32.766 0)
 		(effects
 			(font
